File: kicad/main_board/output.kicad_sch (KiCad schematic)
At the start: 12 parts, among them J12 DRV1, J13 DRV2, J14 CH_IN, J15 CH1, J16 CH2, J17 CH3, J18 CH4

Commit message: remove BAT_INT
Parts:
- renumbered R83 to R82
Changed lines of the file:
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@@
 		(on_board yes)
 		(dnp no)
-		(property "Reference" "#PWR0179"
+		(property "Reference" "#PWR0178"
 			(at 111.76 147.32 0)
 			(effects
@@
 			(project "main_board"
 				(path "/8e1f1504-76c2-49e6-9261-3c1190503f8c/1327ee6b-7a00-44f7-81fe-b42319e4569a"
-					(reference "#PWR0179")
+					(reference "#PWR0178")
 					(unit 1)
 				)
@@
 		(on_board yes)
 		(dnp no)
-		(property "Reference" "#PWR0176"
+		(property "Reference" "#PWR0175"
 			(at 104.14 62.23 0)
 			(effects
@@
 			(project "main_board"
 				(path "/8e1f1504-76c2-49e6-9261-3c1190503f8c/1327ee6b-7a00-44f7-81fe-b42319e4569a"
-					(reference "#PWR0176")
+					(reference "#PWR0175")
 					(unit 1)
 				)
@@
 		(dnp no)
 		(fields_autoplaced yes)
-		(property "Reference" "R83"
+		(property "Reference" "R82"
 			(at 95.25 62.2299 0)
 			(effects
@@
 			(project "main_board"
 				(path "/8e1f1504-76c2-49e6-9261-3c1190503f8c/1327ee6b-7a00-44f7-81fe-b42319e4569a"
-					(reference "R83")
+					(reference "R82")
 					(unit 1)
 				)
@@
 		(on_board yes)
 		(dnp no)
-		(property "Reference" "#PWR0175"
+		(property "Reference" "#PWR0174"
 			(at 92.71 62.23 0)
 			(effects
@@
 			(project "main_board"
 				(path "/8e1f1504-76c2-49e6-9261-3c1190503f8c/1327ee6b-7a00-44f7-81fe-b42319e4569a"
-					(reference "#PWR0175")
+					(reference "#PWR0174")
 					(unit 1)
 				)
@@
 		(on_board yes)
 		(dnp no)
-		(property "Reference" "#PWR0177"
+		(property "Reference" "#PWR0176"
 			(at 111.76 57.15 0)
 			(effects
@@
 			(project "main_board"
 				(path "/8e1f1504-76c2-49e6-9261-3c1190503f8c/1327ee6b-7a00-44f7-81fe-b42319e4569a"
-					(reference "#PWR0177")
+					(reference "#PWR0176")
 					(unit 1)
 				)
@@
 		(on_board yes)
 		(dnp no)
-		(property "Reference" "#PWR0178"
+		(property "Reference" "#PWR0177"
 			(at 111.76 95.25 0)
 			(effects
@@
 			(project "main_board"
 				(path "/8e1f1504-76c2-49e6-9261-3c1190503f8c/1327ee6b-7a00-44f7-81fe-b42319e4569a"
-					(reference "#PWR0178")
-					(unit 1)
-				)
+					(reference "#PWR0177")
+					(unit 1)
+				)

Commit message: update BOM prioritizing basic parts
Parts:
- J12, J13, J14: LCSC (none) -> C2897376
- J15, J16, J17, J18: footprint SaawLib:STX-3100-5N -> SaawLib:PJ-3062-CO; LCSC (none) -> C319113; MOUSER 806-STX-3100-5N -> (none); MPN STX-3100-5N -> (none)
- JP4, JP5, JP6, JP7: LCSC (none) -> C492401
- R82: JLC (none) -> C22935; LCSC C22935 -> (none); MOUSER 603-RC0603FR-071ML -> (none); MPN RC0603FR-071ML -> (none)

Commit message: add generation script
Parts:
- J12, J13, J14, J15, J16, J17, J18, JP4, JP5, JP6, JP7: Service (none) -> HandAssembly
- R82: JLC C22935 -> (none); LCSC (none) -> C22935; Service (none) -> PCBA
Changed lines of the file:
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@@
 			)
 		)
-		(property "JLC" ""
+		(property "Service" "HandAssembly"
 			(at 198.12 104.14 0)
 			(effects
@@
 			)
 		)
-		(property "JLC" ""
+		(property "Service" "HandAssembly"
 			(at 118.11 71.12 0)
 			(effects
@@
 			)
 		)
-		(property "JLC" ""
+		(property "Service" "HandAssembly"
 			(at 118.11 123.19 0)
 			(effects
@@
 			)
 		)
-		(property "JLC" ""
+		(property "Service" "HandAssembly"
 			(at 198.12 129.54 0)
 			(effects
@@
 			)
 		)
-		(property "JLC" ""
+		(property "Service" "HandAssembly"
 			(at 212.09 127 0)
 			(effects
@@
 			)
 		)
-		(property "LCSC" ""
+		(property "LCSC" "C22935"
 			(at 92.71 63.5 0)
 			(effects
@@
 			)
 		)
-		(property "JLC" "C22935"
+		(property "Service" "PCBA"
 			(at 92.71 63.5 0)
 			(effects
@@
 			)
 		)
-		(property "JLC" ""
+		(property "Service" "HandAssembly"
 			(at 179.07 92.71 0)
 			(effects
@@
 			)
 		)
-		(property "JLC" ""
+		(property "Service" "HandAssembly"
 			(at 198.12 55.88 0)
 			(effects
@@
 			)
 		)
-		(property "JLC" ""
+		(property "Service" "HandAssembly"
 			(at 212.09 53.34 0)
 			(effects
@@
 			)
 		)
-		(property "JLC" ""
+		(property "Service" "HandAssembly"
 			(at 198.12 80.01 0)
 			(effects
@@
 			)
 		)
-		(property "JLC" ""
+		(property "Service" "HandAssembly"
 			(at 212.09 77.47 0)
 			(effects
@@
 			)
 		)
-		(property "JLC" ""
+		(property "Service" "HandAssembly"
 			(at 212.09 101.6 0)
 			(effects
