File: kicad/main_board/charger.kicad_sch (KiCad schematic)
At the start: 74 parts, among them J4 BAT, J5 BAT_LINK, Q3 CSD17551Q3A, Q4 CSD17551Q3A, Q5 CSD17551Q3A, Q6 CSD17551Q3A, Q7 CSD25402Q3A, U4 BQ25703A

Commit message: connect charger VBUS before inrush limiter
Parts:
- renumbered R85 to R18, R18 to R19, R84 to R20, R19 to R21, R20 to R22, R21 to R23, R22 to R24, R23 to R25, R24 to R26, R25 to R27, R26 to R28, R27 to R29, R28 to R30, R29 to R31, R87 to R32, R86 to R33, R30 to R34, R31 to R35, R32 to R36, R33 to R37, R34 to R38, R35 to R39
Connections:
- net VCHRG: no longer R28.2
- new net VBUS: R28.2
Changed lines of the file:
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@@
 	(title_block
 		(title "SW32 - Main Board")
-		(date "2024-05-29")
+		(date "2024-05-31")
 		(rev "1")
 		(company "saawsm")
@@
 	)
 	(symbol
+		(lib_id "power:VBUS")
+		(at 114.3 64.77 0)
+		(unit 1)
+		(exclude_from_sim no)
+		(in_bom yes)
+		(on_board yes)
+		(dnp no)
+		(property "Reference" "#PWR046"
+			(at 114.3 68.58 0)
+			(effects
+				(font
+					(size 1.27 1.27)
+				)
+				(hide yes)
+			)
+		)
+		(property "Value" "VBUS"
+			(at 114.3 60.96 0)
+			(effects
+				(font
+					(size 1.27 1.27)
+				)
+			)
+		)
+		(property "Footprint" ""
+			(at 114.3 64.77 0)
+			(effects
+				(font
+					(size 1.27 1.27)
+				)
+				(hide yes)
+			)
+		)
+		(property "Datasheet" ""
+			(at 114.3 64.77 0)
+			(effects
+				(font
+					(size 1.27 1.27)
+				)
+				(hide yes)
+			)
+		)
+		(property "Description" "Power symbol creates a global label with name \"VBUS\""
+			(at 114.3 64.77 0)
+			(effects
+				(font
+					(size 1.27 1.27)
+				)
+				(hide yes)
+			)
+		)
+		(pin "1"
+		)
+		(instances
+			(project "main_board"
+				(path "/8e1f1504-76c2-49e6-9261-3c1190503f8c/1076a657-0b13-48f5-b500-e72d30eb3a1f"
+					(reference "#PWR046")
+					(unit 1)
+				)
+			)
+		)
+	)
+	(symbol
 		(lib_id "Device:C")
 		(at 246.38 27.94 0)
@@
 		(on_board yes)
 		(dnp no)
-		(property "Reference" "R18"
+		(property "Reference" "R19"
 			(at 33.274 113.03 0)
 			(effects
@@
 			(project "main_board"
 				(path "/8e1f1504-76c2-49e6-9261-3c1190503f8c/1076a657-0b13-48f5-b500-e72d30eb3a1f"
-					(reference "R18")
+					(reference "R19")
 					(unit 1)
 				)
@@
 		(on_board yes)
 		(dnp no)
-		(property "Reference" "R28"
+		(property "Reference" "R30"
 			(at 143.764 179.07 0)
 			(effects
@@
 			(project "main_board"
 				(path "/8e1f1504-76c2-49e6-9261-3c1190503f8c/1076a657-0b13-48f5-b500-e72d30eb3a1f"
-					(reference "R28")
+					(reference "R30")
 					(unit 1)
 				)
@@
 		(on_board yes)
 		(dnp no)
-		(property "Reference" "R85"
+		(property "Reference" "R18"
 			(at 33.274 105.41 0)
 			(effects
@@
 			(project "main_board"
 				(path "/8e1f1504-76c2-49e6-9261-3c1190503f8c/1076a657-0b13-48f5-b500-e72d30eb3a1f"
-					(reference "R85")
+					(reference "R18")
 					(unit 1)
 				)
@@
 		(on_board yes)
 		(dnp no)
-		(property "Reference" "R19"
+		(property "Reference" "R21"
 			(at 33.274 152.4 0)
 			(effects
@@
 			(project "main_board"
 				(path "/8e1f1504-76c2-49e6-9261-3c1190503f8c/1076a657-0b13-48f5-b500-e72d30eb3a1f"
-					(reference "R19")
+					(reference "R21")
 					(unit 1)
 				)
@@
 		(on_board yes)
 		(dnp no)
-		(property "Reference" "R35"
+		(property "Reference" "R39"
 			(at 258.064 128.27 0)
 			(effects
@@
 			(project "main_board"
 				(path "/8e1f1504-76c2-49e6-9261-3c1190503f8c/1076a657-0b13-48f5-b500-e72d30eb3a1f"
-					(reference "R35")
+					(reference "R39")
 					(unit 1)
 				)
@@
 		(on_board yes)
 		(dnp no)
-		(property "Reference" "R31"
+		(property "Reference" "R35"
 			(at 236.22 50.292 90)
 			(effects
@@
 			(project "main_board"
 				(path "/8e1f1504-76c2-49e6-9261-3c1190503f8c/1076a657-0b13-48f5-b500-e72d30eb3a1f"
-					(reference "R31")
+					(reference "R35")
 					(unit 1)
 				)
@@
 		(on_board yes)
 		(dnp no)
-		(property "Reference" "R30"
+		(property "Reference" "R34"
 			(at 232.918 78.74 0)
 			(effects
@@
 			(project "main_board"
 				(path "/8e1f1504-76c2-49e6-9261-3c1190503f8c/1076a657-0b13-48f5-b500-e72d30eb3a1f"
-					(reference "R30")
+					(reference "R34")
 					(unit 1)
 				)
@@
 		(on_board yes)
 		(dnp no)
-		(property "Reference" "R86"
+		(property "Reference" "R33"
 			(at 223.774 151.13 0)
 			(effects
@@
 			(project "main_board"
 				(path "/8e1f1504-76c2-49e6-9261-3c1190503f8c/1076a657-0b13-48f5-b500-e72d30eb3a1f"
-					(reference "R86")
+					(reference "R33")
 					(unit 1)
 				)
@@
 		(on_board yes)
 		(dnp no)
-		(property "Reference" "R25"
+		(property "Reference" "R27"
 			(at 87.884 60.96 0)
 			(effects
@@
 			(project "main_board"
 				(path "/8e1f1504-76c2-49e6-9261-3c1190503f8c/1076a657-0b13-48f5-b500-e72d30eb3a1f"
-					(reference "R25")
+					(reference "R27")
 					(unit 1)
 				)
@@
 		(on_board yes)
 		(dnp no)
-		(property "Reference" "R29"
+		(property "Reference" "R31"
 			(at 223.774 135.89 0)
 			(effects
@@
 			(project "main_board"
 				(path "/8e1f1504-76c2-49e6-9261-3c1190503f8c/1076a657-0b13-48f5-b500-e72d30eb3a1f"
-					(reference "R29")
+					(reference "R31")
 					(unit 1)
 				)
@@
 		(on_board yes)
 		(dnp no)
-		(property "Reference" "R23"
+		(property "Reference" "R25"
 			(at 80.01 50.292 90)
 			(effects
@@
 			(project "main_board"
 				(path "/8e1f1504-76c2-49e6-9261-3c1190503f8c/1076a657-0b13-48f5-b500-e72d30eb3a1f"
-					(reference "R23")
+					(reference "R25")
 					(unit 1)
 				)
@@
 		(on_board yes)
 		(dnp no)
-		(property "Reference" "R33"
+		(property "Reference" "R37"
 			(at 258.064 107.95 0)
 			(effects
@@
 			(project "main_board"
 				(path "/8e1f1504-76c2-49e6-9261-3c1190503f8c/1076a657-0b13-48f5-b500-e72d30eb3a1f"
-					(reference "R33")
+					(reference "R37")
 					(unit 1)
 				)
@@
 	)
 	(symbol
-		(lib_id "power:VBUS")
-		(at 114.3 64.77 0)
-		(unit 1)
-		(exclude_from_sim no)
-		(in_bom yes)
-		(on_board yes)
-		(dnp no)
-		(property "Reference" "#PWR046"
-			(at 114.3 68.58 0)
-			(effects
-				(font
-					(size 1.27 1.27)
-				)
-				(hide yes)
-			)
-		)
-		(property "Value" "VCHRG"
-			(at 114.3 60.96 0)
-			(effects
-				(font
-					(size 1.27 1.27)
-				)
-			)
-		)
-		(property "Footprint" ""
-			(at 114.3 64.77 0)
-			(effects
-				(font
-					(size 1.27 1.27)
-				)
-				(hide yes)
-			)
-		)
-		(property "Datasheet" ""
-			(at 114.3 64.77 0)
-			(effects
-				(font
-					(size 1.27 1.27)
-				)
-				(hide yes)
-			)
-		)
-		(property "Description" "Power symbol creates a global label with name \"VCHG_IN\""
-			(at 114.3 64.77 0)
-			(effects
-				(font
-					(size 1.27 1.27)
-				)
-				(hide yes)
-			)
-		)
-		(pin "1"
-		)
-		(instances
-			(project "main_board"
-				(path "/8e1f1504-76c2-49e6-9261-3c1190503f8c/1076a657-0b13-48f5-b500-e72d30eb3a1f"
-					(reference "#PWR046")
-					(unit 1)
-				)
-			)
-		)
-	)
-	(symbol
 		(lib_id "power:+3.3V")
 		(at 245.11 218.44 0)
@@
 		(on_board yes)
 		(dnp no)
-		(property "Reference" "R21"
+		(property "Reference" "R23"
 			(at 49.784 107.95 0)
 			(effects
@@
 			(project "main_board"
 				(path "/8e1f1504-76c2-49e6-9261-3c1190503f8c/1076a657-0b13-48f5-b500-e72d30eb3a1f"
-					(reference "R21")
+					(reference "R23")
 					(unit 1)
 				)
@@
 		(on_board yes)
 		(dnp no)
-		(property "Reference" "R22"
+		(property "Reference" "R24"
 			(at 75.184 60.96 0)
 			(effects
@@
 			(project "main_board"
 				(path "/8e1f1504-76c2-49e6-9261-3c1190503f8c/1076a657-0b13-48f5-b500-e72d30eb3a1f"
-					(reference "R22")
+					(reference "R24")
 					(unit 1)
 				)
@@
 		(on_board yes)
 		(dnp no)
-		(property "Reference" "R34"
+		(property "Reference" "R38"
 			(at 258.064 118.11 0)
 			(effects
@@
 			(project "main_board"
 				(path "/8e1f1504-76c2-49e6-9261-3c1190503f8c/1076a657-0b13-48f5-b500-e72d30eb3a1f"
-					(reference "R34")
+					(reference "R38")
 					(unit 1)
 				)
@@
 		(on_board yes)
 		(dnp no)
-		(property "Reference" "R27"
+		(property "Reference" "R29"
 			(at 119.634 180.34 0)
 			(effects
@@
 			(project "main_board"
 				(path "/8e1f1504-76c2-49e6-9261-3c1190503f8c/1076a657-0b13-48f5-b500-e72d30eb3a1f"
-					(reference "R27")
+					(reference "R29")
 					(unit 1)
 				)
@@
 		(on_board yes)
 		(dnp no)
-		(property "Reference" "R20"
+		(property "Reference" "R22"
 			(at 33.274 162.56 0)
 			(effects
@@
 			(project "main_board"
 				(path "/8e1f1504-76c2-49e6-9261-3c1190503f8c/1076a657-0b13-48f5-b500-e72d30eb3a1f"
-					(reference "R20")
+					(reference "R22")
 					(unit 1)
 				)
@@
 		(on_board yes)
 		(dnp no)
-		(property "Reference" "R24"
+		(property "Reference" "R26"
 			(at 80.01 111.76 90)
 			(effects
@@
 			(project "main_board"
 				(path "/8e1f1504-76c2-49e6-9261-3c1190503f8c/1076a657-0b13-48f5-b500-e72d30eb3a1f"
-					(reference "R24")
+					(reference "R26")
 					(unit 1)
 				)
@@
 		(on_board yes)
 		(dnp no)
-		(property "Reference" "R26"
+		(property "Reference" "R28"
 			(at 116.078 68.58 0)
 			(effects
@@
 			(project "main_board"
 				(path "/8e1f1504-76c2-49e6-9261-3c1190503f8c/1076a657-0b13-48f5-b500-e72d30eb3a1f"
-					(reference "R26")
+					(reference "R28")
 					(unit 1)
 				)
@@
 		(on_board yes)
 		(dnp no)
-		(property "Reference" "R32"
+		(property "Reference" "R36"
 			(at 243.078 78.74 0)
 			(effects
@@
 			(project "main_board"
 				(path "/8e1f1504-76c2-49e6-9261-3c1190503f8c/1076a657-0b13-48f5-b500-e72d30eb3a1f"
-					(reference "R32")
+					(reference "R36")
 					(unit 1)
 				)
@@
 		(on_board yes)
 		(dnp no)
-		(property "Reference" "R84"
+		(property "Reference" "R20"
 			(at 33.782 144.78 0)
 			(effects
@@
 			(project "main_board"
 				(path "/8e1f1504-76c2-49e6-9261-3c1190503f8c/1076a657-0b13-48f5-b500-e72d30eb3a1f"
-					(reference "R84")
+					(reference "R20")
 					(unit 1)
 				)
@@
 		(on_board yes)
 		(dnp no)
-		(property "Reference" "R87"
+		(property "Reference" "R32"
 			(at 223.774 143.51 0)
 			(effects
@@
 			(project "main_board"
 				(path "/8e1f1504-76c2-49e6-9261-3c1190503f8c/1076a657-0b13-48f5-b500-e72d30eb3a1f"
-					(reference "R87")
+					(reference "R32")
 					(unit 1)
 				)
