File: kicad/main_board/charger.kicad_sch (KiCad schematic)
At the start: 74 parts, among them J4 BAT, J5 BAT_LINK, Q3 CSD17551Q3A, Q4 CSD17551Q3A, Q5 CSD17551Q3A, Q6 CSD17551Q3A, Q7 CSD25402Q3A, U4 BQ25703A

Commit message: add mainboard pcb
Parts:
- removed R29: 10k, Resistor_SMD:R_0603_1608Metric, symbol Device:R
- removed TP7: CHRG_OK, TestPoint:TestPoint_Pad_D1.0mm, symbol Connector:TestPoint_Small
- removed TP8: ~{PROCHOT}, TestPoint:TestPoint_Pad_D1.0mm, symbol Connector:TestPoint_Small
- renumbered R30 to R29, R31 to R30, R32 to R31, R33 to R32, R34 to R33, R35 to R34, R36 to R35, R37 to R36, R38 to R37, R39 to R38, TP6 to TP5, TP9 to TP6, TP10 to TP7, TP11 to TP8, TP12 to TP9
Connections:
- net CHRG_OK: no longer names the net of U4.4 (CHRG_OK)
- no-connect marks 3 -> 5

Commit message: use thermal via footprints
Parts:
- Q3, Q4, Q5, Q6, Q7: footprint Package_SON:VSON-8_3.3x3.3mm_P0.65mm_NexFET -> SaawLib:VSON-8_3.3x3.3mm_P0.65mm_NexFET_ThermalVias
Changed lines of the file:
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@@
 	(title_block
 		(title "SW32 - Main Board")
-		(date "2024-06-09")
+		(date "2024-06-11")
 		(rev "1")
 		(company "saawsm")
@@
 			)
 		)
-		(property "Footprint" "Package_SON:VSON-8_3.3x3.3mm_P0.65mm_NexFET"
+		(property "Footprint" "SaawLib:VSON-8_3.3x3.3mm_P0.65mm_NexFET_ThermalVias"
 			(at 140.97 59.69 0)
 			(effects
@@
 			)
 		)
-		(property "Footprint" "Package_SON:VSON-8_3.3x3.3mm_P0.65mm_NexFET"
+		(property "Footprint" "SaawLib:VSON-8_3.3x3.3mm_P0.65mm_NexFET_ThermalVias"
 			(at 207.391 28.067 0)
 			(effects
@@
 			)
 		)
-		(property "Footprint" "Package_SON:VSON-8_3.3x3.3mm_P0.65mm_NexFET"
+		(property "Footprint" "SaawLib:VSON-8_3.3x3.3mm_P0.65mm_NexFET_ThermalVias"
 			(at 123.19 53.34 0)
 			(effects
@@
 			)
 		)
-		(property "Footprint" "Package_SON:VSON-8_3.3x3.3mm_P0.65mm_NexFET"
+		(property "Footprint" "SaawLib:VSON-8_3.3x3.3mm_P0.65mm_NexFET_ThermalVias"
 			(at 173.99 59.69 0)
 			(effects
@@
 			)
 		)
-		(property "Footprint" "Package_SON:VSON-8_3.3x3.3mm_P0.65mm_NexFET"
+		(property "Footprint" "SaawLib:VSON-8_3.3x3.3mm_P0.65mm_NexFET_ThermalVias"
 			(at 191.77 53.34 0)
 			(effects

Commit message: fix title block
Other:
- title: SW32 - Main Board -> SW32
Changed lines of the file:
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@@
 	(paper "A4")
 	(title_block
-		(title "SW32 - Main Board")
-		(date "2024-06-11")
+		(title "SW32")
+		(date "2024-06-12")
 		(rev "1")
 		(company "saawsm")

Commit message: add battery connector part number
Parts:
- J4: LCSC (none) -> C428721
Changed lines of the file:
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@@
 			)
 		)
-		(property "Datasheet" "~"
+		(property "Datasheet" "https://www.lcsc.com/datasheet/lcsc_datasheet_2304241822_Changzhou-Amass-Elec-XT30UPB-M_C428721.pdf"
 			(at 274.32 58.42 0)
 			(effects
@@
 			)
 		)
-		(property "LCSC" ""
+		(property "LCSC" "C428721"
 			(at 274.32 58.42 0)
 			(effects
