File: kicad/main_board/main_board.kicad_pcb (KiCad board)
At the start: 4 copper layers, 198.1 x 61 mm, 271 parts, among them J1 USB_C, J10 LINE_ALT, J11 LINE, J12 DRV, J13 DRV_PWR, J14 CH_IN, J15 CH1, J16 CH2, J17 CH3, J18 CH4, J2 TRIG_A, J3 TRIG_B, J4 BAT, J5 BAT_LINK, J6 FRONT_PANEL, J7 I2C, J8 SWD, J9 MIC, Q1 DMP3018SFV, Q10 AO3401A, Q2 AO3400A, Q3 CSD17551Q3A, Q4 CSD17551Q3A, Q5 CSD17551Q3A, Q6 CSD17551Q3A, Q7 CSD25402Q3A, Q8 AO3400A, Q9 DMP3018SFV, SW1 PWR, U1 SRV05-4, U10 MCP4451-503, U11 MCP6002, U12 MCP6002, U2 SRV05-4, U3 FUSB302B, U4 BQ25703A, U5 TPS560430, U6 TPS560430, U7 MCP4728, U8 RP2040, U9 W25Q128JVS, Y1 12MHz

Commit message: use thermal via footprints
Parts:
- Q1, Q9: footprint Package_SON:Diodes_PowerDI3333-8 -> SaawLib:Diodes_PowerDI3333-8_ThermalVias
- Q3, Q4, Q5, Q6, Q7: footprint Package_SON:VSON-8_3.3x3.3mm_P0.65mm_NexFET -> SaawLib:VSON-8_3.3x3.3mm_P0.65mm_NexFET_ThermalVias
- U8: footprint Package_DFN_QFN:QFN-56-1EP_7x7mm_P0.4mm_EP3.2x3.2mm -> SaawLib:QFN-56-1EP_7x7mm_P0.4mm_EP3.2x3.2mm_ThermalVias
Routing:
- net VIN: vias 0 -> 10
- net VCHRG: vias 8 -> 12
- net GND: vias 267 -> 266
- added copper zone on B.Cu, net Net-(Q3-D)
- added copper zone on B.Cu, net Net-(Q4-D)
- added copper zone on B.Cu, net Net-(Q5-D)
- added copper zone on B.Cu, net VSYS
