File: kicad/main_board/audio.kicad_sch (KiCad schematic)
At the start: 60 parts, among them J10 LINE_ALT, J11 LINE, J9 MIC, Q10 AO3401A, U10 MCP4451-503, U11 MCP6002, U12 MCP6002

Commit message: connect charger VBUS before inrush limiter
Parts:
- renumbered R57 to R62, R58 to R63, R59 to R64, R60 to R65, R61 to R66, R62 to R67, R63 to R68, R64 to R69, R65 to R70, R66 to R71, R67 to R72, R68 to R73, R69 to R74, R70 to R75, R71 to R76, R72 to R77, R73 to R78, R74 to R79, R75 to R80, R76 to R81, R77 to R82, R78 to R83, R79 to R84, R80 to R85, R81 to R86
Changed lines of the file:
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@@
 	(title_block
 		(title "SW32 - Main Board")
-		(date "2024-05-29")
+		(date "2024-05-31")
 		(rev "1")
 		(company "saawsm")
@@
 		(on_board yes)
 		(dnp no)
-		(property "Reference" "R72"
+		(property "Reference" "R77"
 			(at 179.324 40.64 0)
 			(effects
@@
 			(project "main_board"
 				(path "/8e1f1504-76c2-49e6-9261-3c1190503f8c/62c05929-ef0a-4f70-9eff-4dad203c33f9"
-					(reference "R72")
+					(reference "R77")
 					(unit 1)
 				)
@@
 		(on_board yes)
 		(dnp no)
-		(property "Reference" "R62"
+		(property "Reference" "R67"
 			(at 84.074 156.21 0)
 			(effects
@@
 			(project "main_board"
 				(path "/8e1f1504-76c2-49e6-9261-3c1190503f8c/62c05929-ef0a-4f70-9eff-4dad203c33f9"
-					(reference "R62")
+					(reference "R67")
 					(unit 1)
 				)
@@
 		(dnp no)
 		(fields_autoplaced yes)
-		(property "Reference" "R75"
+		(property "Reference" "R80"
 			(at 192.786 66.04 0)
 			(effects
@@
 			(project "main_board"
 				(path "/8e1f1504-76c2-49e6-9261-3c1190503f8c/62c05929-ef0a-4f70-9eff-4dad203c33f9"
-					(reference "R75")
+					(reference "R80")
 					(unit 1)
 				)
@@
 		(on_board yes)
 		(dnp no)
-		(property "Reference" "R58"
+		(property "Reference" "R63"
 			(at 44.704 140.97 0)
 			(effects
@@
 			(project "main_board"
 				(path "/8e1f1504-76c2-49e6-9261-3c1190503f8c/62c05929-ef0a-4f70-9eff-4dad203c33f9"
-					(reference "R58")
+					(reference "R63")
 					(unit 1)
 				)
@@
 		(on_board yes)
 		(dnp no)
-		(property "Reference" "R70"
+		(property "Reference" "R75"
 			(at 167.894 71.12 0)
 			(effects
@@
 			(project "main_board"
 				(path "/8e1f1504-76c2-49e6-9261-3c1190503f8c/62c05929-ef0a-4f70-9eff-4dad203c33f9"
-					(reference "R70")
+					(reference "R75")
 					(unit 1)
 				)
@@
 		(on_board yes)
 		(dnp no)
-		(property "Reference" "R57"
+		(property "Reference" "R62"
 			(at 30.734 123.19 0)
 			(effects
@@
 			(project "main_board"
 				(path "/8e1f1504-76c2-49e6-9261-3c1190503f8c/62c05929-ef0a-4f70-9eff-4dad203c33f9"
-					(reference "R57")
+					(reference "R62")
 					(unit 1)
 				)
@@
 		(on_board yes)
 		(dnp no)
-		(property "Reference" "R76"
+		(property "Reference" "R81"
 			(at 213.36 31.75 90)
 			(effects
@@
 			(project "main_board"
 				(path "/8e1f1504-76c2-49e6-9261-3c1190503f8c/62c05929-ef0a-4f70-9eff-4dad203c33f9"
-					(reference "R76")
+					(reference "R81")
 					(unit 1)
 				)
@@
 		(on_board yes)
 		(dnp no)
-		(property "Reference" "R61"
+		(property "Reference" "R66"
 			(at 67.564 151.13 0)
 			(effects
@@
 			(project "main_board"
 				(path "/8e1f1504-76c2-49e6-9261-3c1190503f8c/62c05929-ef0a-4f70-9eff-4dad203c33f9"
-					(reference "R61")
+					(reference "R66")
 					(unit 1)
 				)
@@
 		(on_board yes)
 		(dnp no)
-		(property "Reference" "R77"
+		(property "Reference" "R82"
 			(at 213.36 92.71 90)
 			(effects
@@
 			(project "main_board"
 				(path "/8e1f1504-76c2-49e6-9261-3c1190503f8c/62c05929-ef0a-4f70-9eff-4dad203c33f9"
-					(reference "R77")
+					(reference "R82")
 					(unit 1)
 				)
@@
 		(dnp no)
 		(fields_autoplaced yes)
-		(property "Reference" "R80"
+		(property "Reference" "R85"
 			(at 236.22 46.9899 0)
 			(effects
@@
 			(project "main_board"
 				(path "/8e1f1504-76c2-49e6-9261-3c1190503f8c/62c05929-ef0a-4f70-9eff-4dad203c33f9"
-					(reference "R80")
+					(reference "R85")
 					(unit 1)
 				)
@@
 		(dnp no)
 		(fields_autoplaced yes)
-		(property "Reference" "R74"
+		(property "Reference" "R79"
 			(at 192.786 55.88 0)
 			(effects
@@
 			(project "main_board"
 				(path "/8e1f1504-76c2-49e6-9261-3c1190503f8c/62c05929-ef0a-4f70-9eff-4dad203c33f9"
-					(reference "R74")
+					(reference "R79")
 					(unit 1)
 				)
@@
 		(on_board yes)
 		(dnp no)
-		(property "Reference" "R66"
+		(property "Reference" "R71"
 			(at 143.51 31.75 90)
 			(effects
@@
 			(project "main_board"
 				(path "/8e1f1504-76c2-49e6-9261-3c1190503f8c/62c05929-ef0a-4f70-9eff-4dad203c33f9"
-					(reference "R66")
+					(reference "R71")
 					(unit 1)
 				)
@@
 		(on_board yes)
 		(dnp no)
-		(property "Reference" "R69"
+		(property "Reference" "R74"
 			(at 167.894 60.96 0)
 			(effects
@@
 			(project "main_board"
 				(path "/8e1f1504-76c2-49e6-9261-3c1190503f8c/62c05929-ef0a-4f70-9eff-4dad203c33f9"
-					(reference "R69")
+					(reference "R74")
 					(unit 1)
 				)
@@
 		(dnp no)
 		(fields_autoplaced yes)
-		(property "Reference" "R65"
+		(property "Reference" "R70"
 			(at 123.19 176.5299 0)
 			(effects
@@
 			(project "main_board"
 				(path "/8e1f1504-76c2-49e6-9261-3c1190503f8c/62c05929-ef0a-4f70-9eff-4dad203c33f9"
-					(reference "R65")
+					(reference "R70")
 					(unit 1)
 				)
@@
 		(dnp no)
 		(fields_autoplaced yes)
-		(property "Reference" "R81"
+		(property "Reference" "R86"
 			(at 236.22 107.9499 0)
 			(effects
@@
 			(project "main_board"
 				(path "/8e1f1504-76c2-49e6-9261-3c1190503f8c/62c05929-ef0a-4f70-9eff-4dad203c33f9"
-					(reference "R81")
+					(reference "R86")
 					(unit 1)
 				)
@@
 		(on_board yes)
 		(dnp no)
-		(property "Reference" "R78"
+		(property "Reference" "R83"
 			(at 224.79 31.75 90)
 			(effects
@@
 			(project "main_board"
 				(path "/8e1f1504-76c2-49e6-9261-3c1190503f8c/62c05929-ef0a-4f70-9eff-4dad203c33f9"
-					(reference "R78")
+					(reference "R83")
 					(unit 1)
 				)
@@
 		(on_board yes)
 		(dnp no)
-		(property "Reference" "R64"
+		(property "Reference" "R69"
 			(at 109.22 161.29 90)
 			(effects
@@
 			(project "main_board"
 				(path "/8e1f1504-76c2-49e6-9261-3c1190503f8c/62c05929-ef0a-4f70-9eff-4dad203c33f9"
-					(reference "R64")
+					(reference "R69")
 					(unit 1)
 				)
@@
 		(on_board yes)
 		(dnp no)
-		(property "Reference" "R63"
+		(property "Reference" "R68"
 			(at 97.79 161.29 90)
 			(effects
@@
 			(project "main_board"
 				(path "/8e1f1504-76c2-49e6-9261-3c1190503f8c/62c05929-ef0a-4f70-9eff-4dad203c33f9"
-					(reference "R63")
+					(reference "R68")
 					(unit 1)
 				)
@@
 		(on_board yes)
 		(dnp no)
-		(property "Reference" "R60"
+		(property "Reference" "R65"
 			(at 67.564 140.97 0)
 			(effects
@@
 			(project "main_board"
 				(path "/8e1f1504-76c2-49e6-9261-3c1190503f8c/62c05929-ef0a-4f70-9eff-4dad203c33f9"
-					(reference "R60")
+					(reference "R65")
 					(unit 1)
 				)
@@
 		(on_board yes)
 		(dnp no)
-		(property "Reference" "R71"
+		(property "Reference" "R76"
 			(at 173.99 158.75 90)
 			(effects
@@
 			(project "main_board"
 				(path "/8e1f1504-76c2-49e6-9261-3c1190503f8c/62c05929-ef0a-4f70-9eff-4dad203c33f9"
-					(reference "R71")
+					(reference "R76")
 					(unit 1)
 				)
@@
 		(on_board yes)
 		(dnp no)
-		(property "Reference" "R68"
+		(property "Reference" "R73"
 			(at 147.32 163.83 90)
 			(effects
@@
 			(project "main_board"
 				(path "/8e1f1504-76c2-49e6-9261-3c1190503f8c/62c05929-ef0a-4f70-9eff-4dad203c33f9"
-					(reference "R68")
+					(reference "R73")
 					(unit 1)
 				)
@@
 		(on_board yes)
 		(dnp no)
-		(property "Reference" "R73"
+		(property "Reference" "R78"
 			(at 181.864 91.44 0)
 			(effects
@@
 			(project "main_board"
 				(path "/8e1f1504-76c2-49e6-9261-3c1190503f8c/62c05929-ef0a-4f70-9eff-4dad203c33f9"
-					(reference "R73")
+					(reference "R78")
 					(unit 1)
 				)
@@
 		(on_board yes)
 		(dnp no)
-		(property "Reference" "R59"
+		(property "Reference" "R64"
 			(at 44.704 151.13 0)
 			(effects
@@
 			(project "main_board"
 				(path "/8e1f1504-76c2-49e6-9261-3c1190503f8c/62c05929-ef0a-4f70-9eff-4dad203c33f9"
-					(reference "R59")
+					(reference "R64")
 					(unit 1)
 				)
@@
 		(on_board yes)
 		(dnp no)
-		(property "Reference" "R67"
+		(property "Reference" "R72"
 			(at 143.51 92.71 90)
 			(effects
@@
 			(project "main_board"
 				(path "/8e1f1504-76c2-49e6-9261-3c1190503f8c/62c05929-ef0a-4f70-9eff-4dad203c33f9"
-					(reference "R67")
+					(reference "R72")
 					(unit 1)
 				)
@@
 		(on_board yes)
 		(dnp no)
-		(property "Reference" "R79"
+		(property "Reference" "R84"
 			(at 224.79 92.71 90)
 			(effects
@@
 			(project "main_board"
 				(path "/8e1f1504-76c2-49e6-9261-3c1190503f8c/62c05929-ef0a-4f70-9eff-4dad203c33f9"
-					(reference "R79")
+					(reference "R84")
 					(unit 1)
 				)

Commit message: add mainboard pcb
Parts:
- removed TP30, TP34: GND, TestPoint:TestPoint_Pad_D1.0mm, symbol Connector:TestPoint_Small
- removed TP31: MOP, TestPoint:TestPoint_Pad_D1.0mm, symbol Connector:TestPoint_Small
- removed TP32: ROP, TestPoint:TestPoint_Pad_D1.0mm, symbol Connector:TestPoint_Small
- removed TP33: TOP, TestPoint:TestPoint_Pad_D1.0mm, symbol Connector:TestPoint_Small
- renumbered R62 to R61, R63 to R62, R64 to R63, R65 to R64, R66 to R65, R67 to R66, R68 to R67, R69 to R68, R70 to R69, R71 to R70, R72 to R71, R73 to R72, R74 to R73, R75 to R74, R76 to R75, R77 to R76, R78 to R77, R79 to R78, R80 to R79, R81 to R80, R82 to R81, R83 to R82, R84 to R83, R85 to R84, R86 to R85

Commit message: fix title block
Other:
- title: SW32 - Main Board -> SW32
Changed lines of the file:
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@@
 	(paper "A4")
 	(title_block
-		(title "SW32 - Main Board")
-		(date "2024-06-11")
+		(title "SW32")
+		(date "2024-06-12")
 		(rev "1")
 		(company "saawsm")
