File: kicad/main_board/controller.kicad_sch (KiCad schematic)
At the start: 44 parts, among them J6 FRONT_PANEL, J7 I2C, J8 SWD, U7 MCP4728, U8 RP2040, U9 W25Q128JVP, Y1 12MHz

Commit message: ground TESTEN pin
Connections:
- net GND: now also U8.19 (TESTEN)
- no-connect marks 2 -> 1
Changed lines of the file:
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@@
 	)
 	(no_connect
-		(at 129.54 146.05)
-	)
-	(no_connect
 		(at 255.27 106.68)
 	)
@@
 		)
 	)
+	(wire
+		(pts
+			(xy 128.27 146.05) (xy 129.54 146.05)
+		)
+		(stroke
+			(width 0)
+			(type default)
+		)
+	)
 	(polyline
 		(pts
@@
 	(wire
 		(pts
+			(xy 128.27 147.32) (xy 128.27 146.05)
+		)
+		(stroke
+			(width 0)
+			(type default)
+		)
+	)
+	(wire
+		(pts
 			(xy 128.27 81.28) (xy 128.27 80.01)
 		)
@@
 		(on_board yes)
 		(dnp no)
-		(property "Reference" "#PWR0131"
+		(property "Reference" "#PWR0132"
 			(at 270.51 77.47 0)
 			(effects
@@
 			(project "main_board"
 				(path "/8e1f1504-76c2-49e6-9261-3c1190503f8c/c17fbfa0-81d7-4817-8752-da6de21e6518"
-					(reference "#PWR0131")
+					(reference "#PWR0132")
 					(unit 1)
 				)
@@
 		(on_board yes)
 		(dnp no)
-		(property "Reference" "#PWR0127"
+		(property "Reference" "#PWR0128"
 			(at 257.81 83.82 0)
 			(effects
@@
 			(project "main_board"
 				(path "/8e1f1504-76c2-49e6-9261-3c1190503f8c/c17fbfa0-81d7-4817-8752-da6de21e6518"
-					(reference "#PWR0127")
+					(reference "#PWR0128")
 					(unit 1)
 				)
@@
 		(on_board yes)
 		(dnp no)
-		(property "Reference" "#PWR0128"
+		(property "Reference" "#PWR0129"
 			(at 257.81 114.3 0)
 			(effects
@@
 			(project "main_board"
 				(path "/8e1f1504-76c2-49e6-9261-3c1190503f8c/c17fbfa0-81d7-4817-8752-da6de21e6518"
-					(reference "#PWR0128")
+					(reference "#PWR0129")
 					(unit 1)
 				)
@@
 		(on_board yes)
 		(dnp no)
-		(property "Reference" "#PWR0116"
+		(property "Reference" "#PWR0117"
 			(at 154.94 161.29 0)
 			(effects
@@
 			(project "main_board"
 				(path "/8e1f1504-76c2-49e6-9261-3c1190503f8c/c17fbfa0-81d7-4817-8752-da6de21e6518"
-					(reference "#PWR0116")
+					(reference "#PWR0117")
 					(unit 1)
 				)
@@
 		(on_board yes)
 		(dnp no)
-		(property "Reference" "#PWR0120"
+		(property "Reference" "#PWR0121"
 			(at 209.55 52.07 0)
 			(effects
@@
 			(project "main_board"
 				(path "/8e1f1504-76c2-49e6-9261-3c1190503f8c/c17fbfa0-81d7-4817-8752-da6de21e6518"
-					(reference "#PWR0120")
+					(reference "#PWR0121")
 					(unit 1)
 				)
@@
 		(on_board yes)
 		(dnp no)
-		(property "Reference" "#PWR0130"
+		(property "Reference" "#PWR0131"
 			(at 262.89 45.72 0)
 			(effects
@@
 			(project "main_board"
 				(path "/8e1f1504-76c2-49e6-9261-3c1190503f8c/c17fbfa0-81d7-4817-8752-da6de21e6518"
-					(reference "#PWR0130")
+					(reference "#PWR0131")
 					(unit 1)
 				)
@@
 		(on_board yes)
 		(dnp no)
-		(property "Reference" "#PWR0117"
+		(property "Reference" "#PWR0118"
 			(at 157.48 60.96 0)
 			(effects
@@
 			(project "main_board"
 				(path "/8e1f1504-76c2-49e6-9261-3c1190503f8c/c17fbfa0-81d7-4817-8752-da6de21e6518"
-					(reference "#PWR0117")
+					(reference "#PWR0118")
 					(unit 1)
 				)
@@
 		(on_board yes)
 		(dnp no)
-		(property "Reference" "#PWR0123"
+		(property "Reference" "#PWR0124"
 			(at 238.76 77.47 0)
 			(effects
@@
 			(project "main_board"
 				(path "/8e1f1504-76c2-49e6-9261-3c1190503f8c/c17fbfa0-81d7-4817-8752-da6de21e6518"
-					(reference "#PWR0123")
+					(reference "#PWR0124")
 					(unit 1)
 				)
@@
 		(on_board yes)
 		(dnp no)
-		(property "Reference" "#PWR0121"
+		(property "Reference" "#PWR0122"
 			(at 209.55 74.93 0)
 			(effects
@@
 			(project "main_board"
 				(path "/8e1f1504-76c2-49e6-9261-3c1190503f8c/c17fbfa0-81d7-4817-8752-da6de21e6518"
-					(reference "#PWR0121")
+					(reference "#PWR0122")
 					(unit 1)
 				)
@@
 		(on_board yes)
 		(dnp no)
-		(property "Reference" "#PWR0125"
+		(property "Reference" "#PWR0126"
 			(at 243.84 132.08 0)
 			(effects
@@
 			(project "main_board"
 				(path "/8e1f1504-76c2-49e6-9261-3c1190503f8c/c17fbfa0-81d7-4817-8752-da6de21e6518"
-					(reference "#PWR0125")
+					(reference "#PWR0126")
 					(unit 1)
 				)
@@
 		(on_board yes)
 		(dnp no)
-		(property "Reference" "#PWR0119"
+		(property "Reference" "#PWR0120"
 			(at 196.85 36.83 0)
 			(effects
@@
 			(project "main_board"
 				(path "/8e1f1504-76c2-49e6-9261-3c1190503f8c/c17fbfa0-81d7-4817-8752-da6de21e6518"
-					(reference "#PWR0119")
+					(reference "#PWR0120")
 					(unit 1)
 				)
@@
 		(on_board yes)
 		(dnp no)
-		(property "Reference" "#PWR0115"
+		(property "Reference" "#PWR0116"
 			(at 152.4 180.34 0)
 			(effects
@@
 			(project "main_board"
 				(path "/8e1f1504-76c2-49e6-9261-3c1190503f8c/c17fbfa0-81d7-4817-8752-da6de21e6518"
-					(reference "#PWR0115")
+					(reference "#PWR0116")
 					(unit 1)
 				)
@@
 		(on_board yes)
 		(dnp no)
-		(property "Reference" "#PWR0129"
+		(property "Reference" "#PWR0130"
 			(at 257.81 165.1 0)
 			(effects
@@
 			(project "main_board"
 				(path "/8e1f1504-76c2-49e6-9261-3c1190503f8c/c17fbfa0-81d7-4817-8752-da6de21e6518"
-					(reference "#PWR0129")
+					(reference "#PWR0130")
 					(unit 1)
 				)
@@
 		(on_board yes)
 		(dnp no)
-		(property "Reference" "#PWR0124"
+		(property "Reference" "#PWR0125"
 			(at 238.76 90.17 0)
 			(effects
@@
 			(project "main_board"
 				(path "/8e1f1504-76c2-49e6-9261-3c1190503f8c/c17fbfa0-81d7-4817-8752-da6de21e6518"
-					(reference "#PWR0124")
+					(reference "#PWR0125")
 					(unit 1)
 				)
@@
 		(on_board yes)
 		(dnp no)
-		(property "Reference" "#PWR0122"
+		(property "Reference" "#PWR0123"
 			(at 237.49 57.15 0)
 			(effects
@@
 			(project "main_board"
 				(path "/8e1f1504-76c2-49e6-9261-3c1190503f8c/c17fbfa0-81d7-4817-8752-da6de21e6518"
-					(reference "#PWR0122")
+					(reference "#PWR0123")
 					(unit 1)
 				)
@@
 		(on_board yes)
 		(dnp no)
-		(property "Reference" "#PWR0126"
+		(property "Reference" "#PWR0127"
 			(at 250.19 45.72 0)
 			(effects
@@
 			(project "main_board"
 				(path "/8e1f1504-76c2-49e6-9261-3c1190503f8c/c17fbfa0-81d7-4817-8752-da6de21e6518"
-					(reference "#PWR0126")
+					(reference "#PWR0127")
 					(unit 1)
 				)
@@
 		(dnp no)
 		(fields_autoplaced yes)
-		(property "Reference" "#PWR0118"
+		(property "Reference" "#PWR0119"
 			(at 163.83 180.34 0)
 			(effects
@@
 			(project "main_board"
 				(path "/8e1f1504-76c2-49e6-9261-3c1190503f8c/c17fbfa0-81d7-4817-8752-da6de21e6518"
-					(reference "#PWR0118")
+					(reference "#PWR0119")
 					(unit 1)
 				)
@@
 					(unit 1)
 				)
+			)
+		)
+	)
+	(symbol
+		(lib_id "power:GND")
+		(at 128.27 147.32 0)
+		(unit 1)
+		(exclude_from_sim no)
+		(in_bom yes)
+		(on_board yes)
+		(dnp no)
+		(property "Reference" "#PWR0115"
+			(at 128.27 153.67 0)
+			(effects
+				(font
+					(size 1.27 1.27)
+				)
+				(hide yes)
+			)
+		)
+		(property "Value" "GND"
+			(at 128.27 151.13 0)
+			(effects
+				(font
+					(size 1.27 1.27)
+				)
+			)
+		)
+		(property "Footprint" ""
+			(at 128.27 147.32 0)
+			(effects
+				(font
+					(size 1.27 1.27)
+				)
+				(hide yes)
+			)
+		)
+		(property "Datasheet" ""
+			(at 128.27 147.32 0)
+			(effects
+				(font
+					(size 1.27 1.27)
+				)
+				(hide yes)
+			)
+		)
+		(property "Description" "Power symbol creates a global label with name \"GND\" , ground"
+			(at 128.27 147.32 0)
+			(effects
+				(font
+					(size 1.27 1.27)
+				)
+				(hide yes)
+			)
+		)
+		(pin "1"
+		)
+		(instances
+			(project "main_board"
+				(path "/8e1f1504-76c2-49e6-9261-3c1190503f8c/c17fbfa0-81d7-4817-8752-da6de21e6518"
+					(reference "#PWR0115")
+					(unit 1)
+				)

Commit message: use SOIC package
Parts:
- R61: now not fitted
- U9: value W25Q128JVP -> W25Q128JVS; footprint Package_SON:WSON-8-1EP_6x5mm_P1.27mm_EP3.4x4.3mm -> Package_SO:SOIC-8_5.23x5.23mm_P1.27mm; symbol Memory_Flash:W25Q32JVZP -> Memory_Flash:W25Q128JVS; LCSC C190862 -> C97521
Connections:
- no-connect marks 1 -> 0
Changed lines of the file:
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@@
 		(color 0 0 0 0)
 	)
-	(no_connect
-		(at 255.27 106.68)
-	)
 	(wire
 		(pts
@@
 		(in_bom yes)
 		(on_board yes)
-		(dnp no)
+		(dnp yes)
 		(fields_autoplaced yes)
 		(property "Reference" "R61"
@@
 	)
 	(symbol
-		(lib_id "Memory_Flash:W25Q32JVZP")
+		(lib_id "Memory_Flash:W25Q128JVS")
 		(at 257.81 93.98 0)
 		(mirror y)
@@
 			)
 		)
-		(property "Value" "W25Q128JVP"
+		(property "Value" "W25Q128JVS"
 			(at 248.92 95.2499 0)
 			(effects
@@
 			)
 		)
-		(property "Footprint" "Package_SON:WSON-8-1EP_6x5mm_P1.27mm_EP3.4x4.3mm"
+		(property "Footprint" "Package_SO:SOIC-8_5.23x5.23mm_P1.27mm"
 			(at 257.81 93.98 0)
 			(effects
@@
 			)
 		)
-		(property "Datasheet" "https://www.lcsc.com/datasheet/lcsc_datasheet_2304140030_Winbond-Elec-W25Q128JVPIQ_C190862.pdf"
+		(property "Datasheet" "https://www.lcsc.com/datasheet/lcsc_datasheet_1811142111_Winbond-Elec-W25Q128JVSIQ_C97521.pdf"
 			(at 257.81 96.52 0)
 			(effects
@@
 			)
 		)
-		(property "Description" "128Mb Serial Flash Memory, Standard/Dual/Quad SPI, WSON-8"
+		(property "Description" "128Mb Serial Flash Memory, Standard/Dual/Quad SPI, SOIC-8"
 			(at 257.81 93.98 0)
 			(effects
@@
 			)
 		)
-		(property "LCSC" "C190862"
+		(property "LCSC" "C97521"
 			(at 257.81 93.98 0)
 			(effects
@@
 		(pin "8"
 		)
-		(pin "9"
-		)
 		(pin "7"

Commit message: add mainboard pcb
Parts:
- removed TP23: DSCL, TestPoint:TestPoint_Pad_D1.0mm, symbol Connector:TestPoint_Small
- removed TP24: DSDA, TestPoint:TestPoint_Pad_D1.0mm, symbol Connector:TestPoint_Small
- C65, C66: footprint Capacitor_SMD:C_0603_1608Metric -> Capacitor_SMD:C_0402_1005Metric; LCSC C1644 -> C1548
- R52: renamed from R53; footprint Resistor_SMD:R_0603_1608Metric -> Resistor_SMD:R_0402_1005Metric; LCSC C25190 -> C25100
- R53: renamed from R54; footprint Resistor_SMD:R_0603_1608Metric -> Resistor_SMD:R_0402_1005Metric; LCSC C25190 -> C25100
- R59: renamed from R60; footprint Resistor_SMD:R_0603_1608Metric -> Resistor_SMD:R_0402_1005Metric; LCSC C21190 -> C11702
- renumbered R50 to R49, R51 to R50, R52 to R51, R55 to R54, R56 to R55, R57 to R56, R58 to R57, R59 to R58, R61 to R60, TP22 to TP18, TP25 to TP19, TP26 to TP20, TP27 to TP21, TP28 to TP22, TP29 to TP23
Connections:
- net +3.3V: now also J6.1 (Pin_1); no longer J6.3 (Pin_3)
- net +5V: now also J6.2 (Pin_2); no longer J6.1 (Pin_1)
- net AUDIO_L: now also U8.41 (GPIO29_ADC3); no longer U8.39 (GPIO27_ADC1)
- net BCLK: now also J6.5 (Pin_5), U8.29 (GPIO18); no longer J6.4 (Pin_4), U8.27 (GPIO16)
- net DIN: now also J6.3 (Pin_3), U8.27 (GPIO16); no longer J6.2 (Pin_2), U8.18 (GPIO15)
- net DISCH_EN: now also U8.36 (GPIO24); no longer U8.30 (GPIO19)
- net DRV_EN: now also U8.13 (GPIO10); no longer U8.29 (GPIO18)
- net GND: now also J6.4 (Pin_4); no longer J6.8 (Pin_8)
- net MIC: now also U8.39 (GPIO27_ADC1); no longer U8.41 (GPIO29_ADC3)
- net PWR_CTRL: now also U8.30 (GPIO19); no longer U8.15 (GPIO12)
- net RXD1: now also U8.32 (GPIO21); no longer U8.12 (GPIO9)
- net SCL: now also U8.35 (GPIO23); no longer U8.32 (GPIO21)
- net SCL_DAC: now also U8.12 (GPIO9); no longer U8.14 (GPIO11)
- net SDA: now also U8.34 (GPIO22); no longer U8.31 (GPIO20)
- net SDA_DAC: now also U8.11 (GPIO8); no longer U8.13 (GPIO10)
- net TXD1: now also J6.8 (Pin_8), U8.31 (GPIO20); no longer J6.5 (Pin_5), U8.11 (GPIO8)
- net ~{INT_PD}: now also U8.37 (GPIO25); no longer U8.16 (GPIO13)
- net ~{PIP_EN}: now also U8.14 (GPIO11); no longer U8.17 (GPIO14)
- net ~{TRIG_A1}: now also U8.17 (GPIO14); no longer U8.34 (GPIO22)
- net ~{TRIG_A2}: now also U8.18 (GPIO15); no longer U8.35 (GPIO23)
- net ~{TRIG_B1}: now also U8.15 (GPIO12); no longer U8.36 (GPIO24)
- net ~{TRIG_B2}: now also U8.16 (GPIO13); no longer U8.37 (GPIO25)

Commit message: use thermal via footprints
Parts:
- U8: footprint Package_DFN_QFN:QFN-56-1EP_7x7mm_P0.4mm_EP3.2x3.2mm -> SaawLib:QFN-56-1EP_7x7mm_P0.4mm_EP3.2x3.2mm_ThermalVias
Changed lines of the file:
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@@
 	(title_block
 		(title "SW32 - Main Board")
-		(date "2024-06-09")
+		(date "2024-06-11")
 		(rev "1")
 		(company "saawsm")
@@
 			)
 		)
-		(property "Footprint" "Package_DFN_QFN:QFN-56-1EP_7x7mm_P0.4mm_EP3.2x3.2mm"
+		(property "Footprint" "SaawLib:QFN-56-1EP_7x7mm_P0.4mm_EP3.2x3.2mm_ThermalVias"
 			(at 154.94 107.95 0)
 			(effects

Commit message: fix title block
Other:
- title: SW32 - Main Board -> SW32
Changed lines of the file:
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@@
 	(paper "A4")
 	(title_block
-		(title "SW32 - Main Board")
-		(date "2024-06-11")
+		(title "SW32")
+		(date "2024-06-12")
 		(rev "1")
 		(company "saawsm")
