File: kicad/main_board/input.kicad_sch (KiCad schematic)
At the start: 37 parts, among them J1 USB_C, J2 TRIG_A, J3 TRIG_B, Q1 DMP3018SFV, Q2 AO3400A, U1 SRV05-4, U2 SRV05-4, U3 FUSB302B

Commit message: add mainboard pcb
Parts:
- removed TP2: GND, TestPoint:TestPoint_Pad_D1.0mm, symbol Connector:TestPoint_Small
- renumbered TP3 to TP2, TP4 to TP3, TP5 to TP4
Connections:
- net CC1: now also U1.6 (IO4); no longer U1.4 (IO3)
- net CC2: now also U1.4 (IO3); no longer U1.6 (IO4)
- net USB_D+: now also U1.3 (IO2); no longer U1.1 (IO1)
- net USB_D-: now also U1.1 (IO1); no longer U1.3 (IO2)

Commit message: use thermal via footprints
Parts:
- Q1: footprint Package_SON:Diodes_PowerDI3333-8 -> SaawLib:Diodes_PowerDI3333-8_ThermalVias
Changed lines of the file:
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@@
 	(title_block
 		(title "SW32 - Main Board")
-		(date "2024-06-09")
+		(date "2024-06-11")
 		(rev "1")
 		(company "saawsm")
@@
 			)
 		)
-		(property "Footprint" "Package_SON:Diodes_PowerDI3333-8"
+		(property "Footprint" "SaawLib:Diodes_PowerDI3333-8_ThermalVias"
 			(at 226.695 34.29 0)
 			(effects

Commit message: fix title block
Other:
- title: SW32 - Main Board -> SW32
Changed lines of the file:
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@@
 	(paper "A4")
 	(title_block
-		(title "SW32 - Main Board")
-		(date "2024-06-11")
+		(title "SW32")
+		(date "2024-06-12")
 		(rev "1")
 		(company "saawsm")
