File: kicad/main_board/power.kicad_sch (KiCad schematic)
At the start: 42 parts, among them Q8 AO3400A, Q9 DMP3018SFV, SW1 SW_Push, U5 TPS560430, U6 TPS560430

Commit message: add inductor footprint
Parts:
- L2, L3: footprint (none) -> SaawLib:L_FNR6028S
Changed lines of the file:
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@@
 			)
 		)
-		(property "Footprint" ""
+		(property "Footprint" "SaawLib:L_FNR6028S"
 			(at 246.38 129.54 0)
 			(effects
@@
 			)
 		)
-		(property "Footprint" ""
+		(property "Footprint" "SaawLib:L_FNR6028S"
 			(at 245.11 50.8 0)
 			(effects

Commit message: use SWPA6020S inductor
Parts:
- L2, L3: footprint SaawLib:L_FNR6028S -> Inductor_SMD:L_Sunlord_SWPA6020S; LCSC C168035 -> C96927
Changed lines of the file:
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@@
 			)
 		)
-		(property "Footprint" "SaawLib:L_FNR6028S"
+		(property "Footprint" "Inductor_SMD:L_Sunlord_SWPA6020S"
 			(at 246.38 129.54 0)
 			(effects
@@
 			)
 		)
-		(property "Datasheet" "https://www.lcsc.com/datasheet/lcsc_datasheet_2304140030_cjiang--Changjiang-Microelectronics-Tech-FNR6028S120MT_C168035.pdf"
+		(property "Datasheet" "https://www.lcsc.com/datasheet/lcsc_datasheet_2310251551_Sunlord-SWPA6020S120MT_C96927.pdf"
 			(at 246.38 129.54 0)
 			(effects
@@
 			)
 		)
-		(property "LCSC" "C168035"
+		(property "LCSC" "C96927"
 			(at 246.38 129.54 0)
 			(effects
@@
 			)
 		)
-		(property "Footprint" "SaawLib:L_FNR6028S"
+		(property "Footprint" "Inductor_SMD:L_Sunlord_SWPA6020S"
 			(at 245.11 50.8 0)
 			(effects
@@
 			)
 		)
-		(property "Datasheet" "https://www.lcsc.com/datasheet/lcsc_datasheet_2304140030_cjiang--Changjiang-Microelectronics-Tech-FNR6028S120MT_C168035.pdf"
+		(property "Datasheet" "https://www.lcsc.com/datasheet/lcsc_datasheet_2310251551_Sunlord-SWPA6020S120MT_C96927.pdf"
 			(at 245.11 50.8 0)
 			(effects
@@
 			)
 		)
-		(property "LCSC" "C168035"
+		(property "LCSC" "C96927"
 			(at 245.11 50.8 0)
 			(effects

Commit message: add VBUS tvs
Parts:
- SW1: value SW_Push -> PWR
Changed lines of the file:
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@@
 			)
 		)
-		(property "Value" "SW_Push"
+		(property "Value" "PWR"
 			(at 88.9 114.2999 90)
 			(effects

Commit message: connect charger VBUS before inrush limiter
Parts:
- renumbered R36 to R40, R37 to R41, R38 to R42, R39 to R43, R40 to R44, R41 to R45, R83 to R46, R42 to R47, R43 to R48, R44 to R49
Changed lines of the file:
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@@
 	(title_block
 		(title "SW32 - Main Board")
-		(date "2024-05-29")
+		(date "2024-05-31")
 		(rev "1")
 		(company "saawsm")
@@
 		(on_board yes)
 		(dnp no)
-		(property "Reference" "R41"
+		(property "Reference" "R45"
 			(at 254.762 54.61 0)
 			(effects
@@
 			(project "main_board"
 				(path "/8e1f1504-76c2-49e6-9261-3c1190503f8c/afe2ed97-1c60-4e5a-9a63-45f783bd4ddb"
-					(reference "R41")
+					(reference "R45")
 					(unit 1)
 				)
@@
 		(on_board yes)
 		(dnp no)
-		(property "Reference" "R42"
+		(property "Reference" "R47"
 			(at 254.762 72.39 0)
 			(effects
@@
 			(project "main_board"
 				(path "/8e1f1504-76c2-49e6-9261-3c1190503f8c/afe2ed97-1c60-4e5a-9a63-45f783bd4ddb"
-					(reference "R42")
+					(reference "R47")
 					(unit 1)
 				)
@@
 		(on_board yes)
 		(dnp no)
-		(property "Reference" "R83"
+		(property "Reference" "R46"
 			(at 254.762 62.23 0)
 			(effects
@@
 			(project "main_board"
 				(path "/8e1f1504-76c2-49e6-9261-3c1190503f8c/afe2ed97-1c60-4e5a-9a63-45f783bd4ddb"
-					(reference "R83")
+					(reference "R46")
 					(unit 1)
 				)
@@
 		(on_board yes)
 		(dnp no)
-		(property "Reference" "R44"
+		(property "Reference" "R49"
 			(at 256.032 143.51 0)
 			(effects
@@
 			(project "main_board"
 				(path "/8e1f1504-76c2-49e6-9261-3c1190503f8c/afe2ed97-1c60-4e5a-9a63-45f783bd4ddb"
-					(reference "R44")
+					(reference "R49")
 					(unit 1)
 				)
@@
 		(on_board yes)
 		(dnp no)
-		(property "Reference" "R38"
+		(property "Reference" "R42"
 			(at 94.742 147.32 0)
 			(effects
@@
 			(project "main_board"
 				(path "/8e1f1504-76c2-49e6-9261-3c1190503f8c/afe2ed97-1c60-4e5a-9a63-45f783bd4ddb"
-					(reference "R38")
+					(reference "R42")
 					(unit 1)
 				)
@@
 		(on_board yes)
 		(dnp no)
-		(property "Reference" "R37"
+		(property "Reference" "R41"
 			(at 58.42 99.06 90)
 			(effects
@@
 			(project "main_board"
 				(path "/8e1f1504-76c2-49e6-9261-3c1190503f8c/afe2ed97-1c60-4e5a-9a63-45f783bd4ddb"
-					(reference "R37")
+					(reference "R41")
 					(unit 1)
 				)
@@
 		(on_board yes)
 		(dnp no)
-		(property "Reference" "R36"
+		(property "Reference" "R40"
 			(at 41.91 138.43 90)
 			(effects
@@
 			(project "main_board"
 				(path "/8e1f1504-76c2-49e6-9261-3c1190503f8c/afe2ed97-1c60-4e5a-9a63-45f783bd4ddb"
-					(reference "R36")
+					(reference "R40")
 					(unit 1)
 				)
@@
 		(on_board yes)
 		(dnp no)
-		(property "Reference" "R39"
+		(property "Reference" "R43"
 			(at 106.172 60.96 0)
 			(effects
@@
 			(project "main_board"
 				(path "/8e1f1504-76c2-49e6-9261-3c1190503f8c/afe2ed97-1c60-4e5a-9a63-45f783bd4ddb"
-					(reference "R39")
+					(reference "R43")
 					(unit 1)
 				)
@@
 		(on_board yes)
 		(dnp no)
-		(property "Reference" "R40"
+		(property "Reference" "R44"
 			(at 163.576 176.53 0)
 			(effects
@@
 			(project "main_board"
 				(path "/8e1f1504-76c2-49e6-9261-3c1190503f8c/afe2ed97-1c60-4e5a-9a63-45f783bd4ddb"
-					(reference "R40")
+					(reference "R44")
 					(unit 1)
 				)
@@
 		(on_board yes)
 		(dnp no)
-		(property "Reference" "R43"
+		(property "Reference" "R48"
 			(at 256.032 133.35 0)
 			(effects
@@
 			(project "main_board"
 				(path "/8e1f1504-76c2-49e6-9261-3c1190503f8c/afe2ed97-1c60-4e5a-9a63-45f783bd4ddb"
-					(reference "R43")
+					(reference "R48")
 					(unit 1)
 				)

Commit message: add mainboard pcb
Parts:
- removed TP13: VIN, TestPoint:TestPoint_Pad_D1.0mm, symbol Connector:TestPoint_Small
- renumbered R40 to R39, R41 to R40, R42 to R41, R43 to R42, R44 to R43, R45 to R44, R46 to R45, R47 to R46, R48 to R47, R49 to R48, TP14 to TP10, TP15 to TP11, TP16 to TP12, TP17 to TP13, TP18 to TP14, TP19 to TP15, TP20 to TP16, TP21 to TP17

Commit message: use thermal via footprints
Parts:
- Q9: footprint Package_SON:Diodes_PowerDI3333-8 -> SaawLib:Diodes_PowerDI3333-8_ThermalVias
Changed lines of the file:
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@@
 	(title_block
 		(title "SW32 - Main Board")
-		(date "2024-06-09")
+		(date "2024-06-11")
 		(rev "1")
 		(company "saawsm")
@@
 			)
 		)
-		(property "Footprint" "Package_SON:Diodes_PowerDI3333-8"
+		(property "Footprint" "SaawLib:Diodes_PowerDI3333-8_ThermalVias"
 			(at 116.205 53.34 0)
 			(effects

Commit message: fix title block
Other:
- title: SW32 - Main Board -> SW32
Changed lines of the file:
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@@
 	(paper "A4")
 	(title_block
-		(title "SW32 - Main Board")
-		(date "2024-06-11")
+		(title "SW32")
+		(date "2024-06-12")
 		(rev "1")
 		(company "saawsm")
