File: kicad/front_control_board/front_control_board.kicad_pcb (KiCad board)
At the start: 2 copper layers, 0 parts

Commit message: add draft front control board pcb
Parts:
- added BZ1: Buzzer, Buzzer_Beeper:Buzzer_12x9.5RM7.6, B.Cu at (170.7, 91.9)
- added C1: 100nF, Capacitor_SMD:C_0603_1608Metric, F.Cu at (174.8, 101.3)
- added C10: 100nF, Capacitor_SMD:C_0603_1608Metric, F.Cu at (188.2, 127.4)
- added C11: 100nF, Capacitor_SMD:C_0603_1608Metric, F.Cu at (206.0, 127.4)
- added C12: 100nF, Capacitor_SMD:C_0603_1608Metric, F.Cu at (223.8, 127.4)
- added C13: 100nF, Capacitor_SMD:C_0603_1608Metric, F.Cu at (241.6, 127.4)
- added C14: 100nF, Capacitor_SMD:C_0603_1608Metric, F.Cu at (172.3, 105.0)
- added C15: 100nF, Capacitor_SMD:C_0603_1608Metric, F.Cu at (174.8, 105.0)
- added C16: 100nF, Capacitor_SMD:C_0603_1608Metric, F.Cu at (174.8, 108.7)
- added C17: 100nF, Capacitor_SMD:C_0603_1608Metric, F.Cu at (172.3, 108.7)
- added C2: 100nF, Capacitor_SMD:C_0603_1608Metric, F.Cu at (217.4, 102.9)
- added C3: 100nF, Capacitor_SMD:C_0603_1608Metric, F.Cu at (62.9, 120.7)
- added C4: 10uF, Capacitor_SMD:C_0603_1608Metric, F.Cu at (172.3, 101.3)
- added C5: 100nF, Capacitor_SMD:C_0603_1608Metric, F.Cu at (94.2, 127.4)
- added C6: 100nF, Capacitor_SMD:C_0603_1608Metric, F.Cu at (119.6, 127.4)
- added C7: 100nF, Capacitor_SMD:C_0603_1608Metric, F.Cu at (134.9, 127.4)
- added C8: 100nF, Capacitor_SMD:C_0603_1608Metric, F.Cu at (152.7, 127.4)
- added C9: 100nF, Capacitor_SMD:C_0603_1608Metric, F.Cu at (167.9, 127.4)
- added D1: PWR, LED_SMD:LED_WS2812B_PLCC4_5.0x5.0mm_P3.2mm, F.Cu at (63.5, 125.7)
- added D10: CH3, LED_SMD:LED_WS2812B_PLCC4_5.0x5.0mm_P3.2mm, F.Cu at (218.4, 125.7)
- added D11: CH4, LED_SMD:LED_WS2812B_PLCC4_5.0x5.0mm_P3.2mm, F.Cu at (236.2, 125.7)
- added D2: 30V, Diode_SMD:D_SOD-323, F.Cu at (67.3, 120.7)
- added D3: USB, LED_SMD:LED_WS2812B_PLCC4_5.0x5.0mm_P3.2mm, F.Cu at (88.9, 125.7)
- added D4: MIC, LED_SMD:LED_WS2812B_PLCC4_5.0x5.0mm_P3.2mm, F.Cu at (114.3, 125.7)
- added D5: LINE, LED_SMD:LED_WS2812B_PLCC4_5.0x5.0mm_P3.2mm, F.Cu at (129.5, 125.7)
- added D6: TRIG_A, LED_SMD:LED_WS2812B_PLCC4_5.0x5.0mm_P3.2mm, F.Cu at (147.3, 125.7)
- added D7: TRIG_B, LED_SMD:LED_WS2812B_PLCC4_5.0x5.0mm_P3.2mm, F.Cu at (162.6, 125.7)
- added D8: CH1, LED_SMD:LED_WS2812B_PLCC4_5.0x5.0mm_P3.2mm, F.Cu at (182.9, 125.7)
- added D9: CH2, LED_SMD:LED_WS2812B_PLCC4_5.0x5.0mm_P3.2mm, F.Cu at (200.7, 125.7)
- added FID1: Fiducial, Fiducial:Fiducial_1mm_Mask2mm, F.Cu at (119.3, 83.9)
- added FID2: Fiducial, Fiducial:Fiducial_1mm_Mask2mm, F.Cu at (245.1, 125.7)
- added FID3: Fiducial, Fiducial:Fiducial_1mm_Mask2mm, F.Cu at (76.7, 122.7)
- added H1: MountingHole, MountingHole:MountingHole_2.2mm_M2, F.Cu at (113.0, 83.8)
- added H2: MountingHole, MountingHole:MountingHole_2.2mm_M2, F.Cu at (245.1, 83.8)
- added H3: MountingHole, MountingHole:MountingHole_2.2mm_M2, F.Cu at (245.1, 113.0)
- added H4: MountingHole, MountingHole:MountingHole_2.2mm_M2, F.Cu at (113.0, 113.0)
- added H5: MountingHole, MountingHole:MountingHole_2.2mm_M2, F.Cu at (72.4, 125.7)
- added J1: MAIN_BOARD, Connector_IDC:IDC-Header_2x04_P2.54mm_Vertical, B.Cu at (145.5, 88.1)
- added J2: PROG, Connector_IDC:IDC-Header_2x03_P2.54mm_Vertical, B.Cu at (212.1, 102.9)
- added J3: DISPLAY, Connector_PinHeader_2.54mm:PinHeader_1x10_P2.54mm_Vertical, B.Cu at (116.7, 109.8)
- added J4: LED_OUT, Connector_PinHeader_2.54mm:PinHeader_1x03_P2.54mm_Vertical, B.Cu at (245.1, 99.1)
- added JP1: BZ1, Jumper:SolderJumper-3_P1.3mm_Bridged12_RoundedPad1.0x1.5mm_NumberLabels, F.Cu at (166.6, 103.1)
- added JP2: BZ2, Jumper:SolderJumper-2_P1.3mm_Bridged_RoundedPad1.0x1.5mm, F.Cu at (173.4, 97.5)
- added Q1: AO3400A, Package_TO_SOT_SMD:SOT-23, F.Cu at (169.2, 97.5)
- added R1: 10k, Resistor_SMD:R_0603_1608Metric, F.Cu at (157.5, 103.6)
- added R10: 10k, Resistor_SMD:R_0603_1608Metric, F.Cu at (145.8, 112.8)
- added R11: 10k, Resistor_SMD:R_0603_1608Metric, F.Cu at (140.7, 112.8)
- added R12: 10k, Resistor_SMD:R_0603_1608Metric, F.Cu at (148.3, 112.8)
- added R13: 10k, Resistor_SMD:R_0603_1608Metric, F.Cu at (143.3, 112.8)
- added R2: 10k, Resistor_SMD:R_0603_1608Metric, F.Cu at (160.0, 103.6)
- added R3: 10k, Resistor_SMD:R_0603_1608Metric, F.Cu at (169.9, 101.3)
- added R4: 10k, Resistor_SMD:R_0603_1608Metric, F.Cu at (154.9, 103.6)
- added R5: 10k, Resistor_SMD:R_0603_1608Metric, F.Cu at (113.0, 99.7)
- added R6: 10k, Resistor_SMD:R_0603_1608Metric, F.Cu at (217.4, 100.3)
- added R7: 10k, Resistor_SMD:R_0603_1608Metric, F.Cu at (113.0, 97.2)
- added R8: 10k, Resistor_SMD:R_0603_1608Metric, F.Cu at (113.0, 104.8)
- added R9: 1k, Resistor_SMD:R_0603_1608Metric, F.Cu at (227.5, 88.8)
- added RV1: CH1, Potentiometer_THT:Potentiometer_Bourns_PTV09A-1_Single_Vertical, F.Cu at (180.4, 84.9)
- added RV2: CH2, Potentiometer_THT:Potentiometer_Bourns_PTV09A-1_Single_Vertical, F.Cu at (198.2, 84.9)
- added RV3: CH3, Potentiometer_THT:Potentiometer_Bourns_PTV09A-1_Single_Vertical, F.Cu at (215.9, 84.9)
- added RV4: CH4, Potentiometer_THT:Potentiometer_Bourns_PTV09A-1_Single_Vertical, F.Cu at (233.7, 84.9)
- added SW1: PEC11R-4215K-S00xx, SaawLib:Rotary_Encoder_Switched_PEC11R, F.Cu at (157.5, 91.9)
- added SW2: BTN1, Button_Switch_THT:SW_PUSH_6mm_H5mm, F.Cu at (119.7, 95.2)
- added SW3: BTN4, Button_Switch_THT:SW_PUSH_6mm_H5mm, F.Cu at (119.7, 108.2)
- added SW4: BTN2, Button_Switch_THT:SW_PUSH_6mm_H5mm, F.Cu at (132.7, 95.2)
- added SW5: BTN3, Button_Switch_THT:SW_PUSH_6mm_H5mm, F.Cu at (132.7, 108.2)
- added U1: ESP32-WROOM-32UE, RF_Module:ESP32-WROOM-32UE, F.Cu at (186.2, 109.2)
Routing:
- net +3.3V: track 0.00 -> 241.9 mm, vias 0 -> 5
- net +5V: track 0.00 -> 201.6 mm
- net /LED_DATA: track 0.00 -> 145.5 mm, vias 0 -> 2
- net /~{LCD_RST/IO0}: track 0.00 -> 125.3 mm, vias 0 -> 2
- net /MOSI: track 0.00 -> 122.8 mm
- net /SCK: track 0.00 -> 119.2 mm, vias 0 -> 2
- net /MISO: track 0.00 -> 113.4 mm
- net /LCD_DC: track 0.00 -> 112.0 mm, vias 0 -> 2
- net /~{LCD_CS}: track 0.00 -> 107.5 mm, vias 0 -> 2
- net /~{CARD_CS}: track 0.00 -> 91.5 mm, vias 0 -> 2
- net /~{BTN4}: track 0.00 -> 90.8 mm, vias 0 -> 1
- net /CH4: track 0.00 -> 86.9 mm, vias 0 -> 2
- net /LCD_LITE: track 0.00 -> 86.0 mm
- net /RXD0: track 0.00 -> 79.8 mm, vias 0 -> 3
- net /TXD0: track 0.00 -> 79.4 mm, vias 0 -> 3
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- added copper zone on F.Cu, net +5V
- added copper zone on B.Cu, net GND
- added copper zone on F.Cu, net GND
Other:
- board outline added: 189.2 x 48.9 mm
- board text added: "1.8{dblquote} TFT Display"
- board text added: "JLCJLCJLCJLC"

Commit message: cleanup
Parts:
- D4: value MIC -> LINE
- D5: value LINE -> MIC
- moved C5 0.64 mm to (94.9, 127.4)
- moved C6 0.64 mm to (120.3, 127.4)
- moved C10 0.63 mm to (188.8, 127.4)
- moved C11 0.63 mm to (206.6, 127.4)
- moved C12 0.63 mm to (224.4, 127.4)
- moved C13 0.63 mm to (242.2, 127.4)
- moved C7 0.63 mm to (135.5, 127.4)
- moved C8 0.63 mm to (153.3, 127.4)
- moved C9 0.63 mm to (168.5, 127.4)
Routing:
- net +5V: track 201.6 -> 207.3 mm
- net GND: vias 46 -> 47

Commit message: add silkscreen board info
Other:
- board text added: "SW32 ${PROJECTNAME} rev${REVISION} ${hash}"
Changed lines of the file:
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@@
+		)
+	)
+	(gr_text "SW32\n${PROJECTNAME} \nrev${REVISION} ${hash}"
+		(locked yes)
+		(at 212.979 112.776 0)
+		(layer "F.SilkS")
+		(effects
+			(font
+				(size 1 1)
+				(thickness 0.15)
+				(bold yes)
+			)
+			(justify left)
 		)
 	)
