File: kicad/front_control_board/front_control_board.kicad_sch (KiCad schematic)
At the start: 67 parts, among them J1 MAIN_BOARD, J2 PROG, J3 DISPLAY, J4 LED_OUT, Q1 AO3400A, SW1 PEC11R-4215K-S00xx, SW2 BTN1, SW3 BTN4, SW4 BTN2, SW5 BTN3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

Commit message: move ground to center pin
Connections:
- net +3.3V: now also J1.1 (Pin_1); no longer J1.3 (Pin_3)
- net +5V: now also J1.2 (Pin_2); no longer J1.1 (Pin_1)
- net BCLK: now also J1.5 (Pin_5); no longer J1.4 (Pin_4)
- net DOUT: now also J1.3 (Pin_3), U1.8 (IO32); no longer J1.2 (Pin_2), U1.10 (IO25)
- net GND: now also J1.4 (Pin_4); no longer J1.8 (Pin_8)
- net RXD0: now also J1.8 (Pin_8); no longer J1.5 (Pin_5)
- net WS: now also U1.10 (IO25); no longer U1.8 (IO32)
Other:
- moved on the sheet: J1
Changed lines of the file:
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@@
 	(wire
 		(pts
-			(xy 36.83 182.88) (xy 35.56 182.88)
-		)
-		(stroke
-			(width 0)
-			(type default)
-		)
-	)
-	(wire
-		(pts
 			(xy 242.57 20.32) (xy 242.57 24.13)
 		)
@@
 	(wire
 		(pts
-			(xy 15.24 177.8) (xy 22.86 177.8)
+			(xy 16.51 175.26) (xy 21.59 175.26)
 		)
 		(stroke
@@
 		)
 	)
-	(wire
-		(pts
-			(xy 36.83 184.15) (xy 36.83 182.88)
-		)
-		(stroke
-			(width 0)
-			(type default)
-		)
-	)
 	(polyline
 		(pts
@@
 	(wire
 		(pts
-			(xy 22.86 180.34) (xy 17.78 180.34)
+			(xy 34.29 182.88) (xy 41.91 182.88)
 		)
 		(stroke
@@
 	(wire
 		(pts
-			(xy 35.56 180.34) (xy 40.64 180.34)
+			(xy 34.29 180.34) (xy 41.91 180.34)
 		)
 		(stroke
@@
 	(wire
 		(pts
-			(xy 35.56 175.26) (xy 40.64 175.26)
+			(xy 21.59 180.34) (xy 16.51 180.34)
 		)
 		(stroke
@@
 	(wire
 		(pts
+			(xy 34.29 177.8) (xy 35.56 177.8)
+		)
+		(stroke
+			(width 0)
+			(type default)
+		)
+	)
+	(wire
+		(pts
 			(xy 270.51 219.71) (xy 270.51 220.98)
 		)
@@
 	(wire
 		(pts
-			(xy 20.32 175.26) (xy 20.32 173.99)
+			(xy 39.37 175.26) (xy 39.37 173.99)
 		)
 		(stroke
@@
 	(wire
 		(pts
+			(xy 35.56 177.8) (xy 35.56 184.15)
+		)
+		(stroke
+			(width 0)
+			(type default)
+		)
+	)
+	(wire
+		(pts
 			(xy 93.98 40.64) (xy 96.52 40.64)
 		)
@@
 	(wire
 		(pts
-			(xy 22.86 182.88) (xy 17.78 182.88)
+			(xy 21.59 182.88) (xy 16.51 182.88)
 		)
 		(stroke
@@
 	(wire
 		(pts
-			(xy 20.32 175.26) (xy 22.86 175.26)
+			(xy 39.37 175.26) (xy 34.29 175.26)
 		)
 		(stroke
@@
 	(wire
 		(pts
-			(xy 15.24 173.99) (xy 15.24 177.8)
+			(xy 16.51 173.99) (xy 16.51 175.26)
 		)
 		(stroke
@@
 	(wire
 		(pts
-			(xy 35.56 177.8) (xy 40.64 177.8)
+			(xy 21.59 177.8) (xy 16.51 177.8)
 		)
 		(stroke
@@
 	(text "3.3V logic"
 		(exclude_from_sim no)
-		(at 25.4 186.944 0)
+		(at 24.13 186.944 0)
 		(effects
 			(font
@@
 	)
 	(label "DOUT"
-		(at 40.64 175.26 180)
+		(at 16.51 177.8 0)
 		(fields_autoplaced yes)
 		(effects
@@
 				(size 1.27 1.27)
 			)
-			(justify right bottom)
+			(justify left bottom)
 		)
 	)
 	(label "BCLK"
-		(at 40.64 177.8 180)
+		(at 16.51 180.34 0)
 		(fields_autoplaced yes)
 		(effects
@@
 				(size 1.27 1.27)
 			)
-			(justify right bottom)
+			(justify left bottom)
 		)
 	)
@@
 	)
 	(label "RXD0"
-		(at 17.78 180.34 0)
+		(at 41.91 182.88 180)
 		(fields_autoplaced yes)
 		(effects
@@
 				(size 1.27 1.27)
 			)
-			(justify left bottom)
+			(justify right bottom)
 		)
 	)
@@
 	)
 	(label "DOUT"
-		(at 157.48 128.27 180)
+		(at 157.48 135.89 180)
 		(fields_autoplaced yes)
 		(effects
@@
 	)
 	(label "TXD0"
-		(at 17.78 182.88 0)
+		(at 16.51 182.88 0)
 		(fields_autoplaced yes)
 		(effects
@@
 	)
 	(label "WS"
-		(at 157.48 135.89 180)
+		(at 157.48 128.27 180)
 		(fields_autoplaced yes)
 		(effects
@@
 	)
 	(label "WS"
-		(at 40.64 180.34 180)
+		(at 41.91 180.34 180)
 		(fields_autoplaced yes)
 		(effects
@@
 	(symbol
 		(lib_id "Connector_Generic:Conn_02x04_Odd_Even")
-		(at 27.94 177.8 0)
+		(at 26.67 177.8 0)
 		(unit 1)
 		(exclude_from_sim no)
@@
 		(fields_autoplaced yes)
 		(property "Reference" "J1"
-			(at 29.21 168.91 0)
+			(at 27.94 168.91 0)
 			(effects
 				(font
@@
 		)
 		(property "Value" "MAIN_BOARD"
-			(at 29.21 171.45 0)
+			(at 27.94 171.45 0)
 			(effects
 				(font
@@
 		)
 		(property "Footprint" "Connector_IDC:IDC-Header_2x04_P2.54mm_Vertical"
-			(at 27.94 177.8 0)
+			(at 26.67 177.8 0)
 			(effects
 				(font
@@
 		)
 		(property "Datasheet" "https://www.lcsc.com/datasheet/lcsc_datasheet_2303141000_HCTL-HC-JN254-2-04-Z_C5372864.pdf"
-			(at 27.94 177.8 0)
+			(at 26.67 177.8 0)
 			(effects
 				(font
@@
 		)
 		(property "Description" "Generic connector, double row, 02x04, odd/even pin numbering scheme (row 1 odd numbers, row 2 even numbers), script generated (kicad-library-utils/schlib/autogen/connector/)"
-			(at 27.94 177.8 0)
+			(at 26.67 177.8 0)
 			(effects
 				(font
@@
 		)
 		(property "LCSC" "C5372864"
-			(at 27.94 177.8 0)
+			(at 26.67 177.8 0)
 			(effects
 				(font
@@
 		)
 		(property "Service" "HandAssembly"
-			(at 27.94 177.8 0)
+			(at 26.67 177.8 0)
 			(effects
 				(font
@@
 	(symbol
 		(lib_id "power:GND")
-		(at 36.83 184.15 0)
+		(at 35.56 184.15 0)
 		(unit 1)
 		(exclude_from_sim no)
@@
 		(dnp no)
 		(property "Reference" "#PWR05"
-			(at 36.83 190.5 0)
+			(at 35.56 190.5 0)
 			(effects
 				(font
@@
 		)
 		(property "Value" "GND"
-			(at 36.83 187.96 0)
+			(at 35.56 187.96 0)
 			(effects
 				(font
@@
 		)
 		(property "Footprint" ""
-			(at 36.83 184.15 0)
+			(at 35.56 184.15 0)
 			(effects
 				(font
@@
 		)
 		(property "Datasheet" ""
-			(at 36.83 184.15 0)
+			(at 35.56 184.15 0)
 			(effects
 				(font
@@
 		)
 		(property "Description" "Power symbol creates a global label with name \"GND\" , ground"
-			(at 36.83 184.15 0)
+			(at 35.56 184.15 0)
 			(effects
 				(font
@@
 	(symbol
 		(lib_id "power:+3.3V")
-		(at 15.24 173.99 0)
+		(at 16.51 173.99 0)
 		(mirror y)
 		(unit 1)
@@
 		(dnp no)
 		(property "Reference" "#PWR01"
-			(at 15.24 177.8 0)
+			(at 16.51 177.8 0)
 			(effects
 				(font
@@
 		)
 		(property "Value" "+3.3V"
-			(at 15.24 170.18 0)
+			(at 16.51 170.18 0)
 			(effects
 				(font
@@
 		)
 		(property "Footprint" ""
-			(at 15.24 173.99 0)
+			(at 16.51 173.99 0)
 			(effects
 				(font
@@
 		)
 		(property "Datasheet" ""
-			(at 15.24 173.99 0)
+			(at 16.51 173.99 0)
 			(effects
 				(font
@@
 		)
 		(property "Description" "Power symbol creates a global label with name \"+3.3V\""
-			(at 15.24 173.99 0)
+			(at 16.51 173.99 0)
 			(effects
 				(font
@@
 	(symbol
 		(lib_id "power:+5V")
-		(at 20.32 173.99 0)
-		(mirror y)
+		(at 39.37 173.99 0)
 		(unit 1)
 		(exclude_from_sim no)
@@
 		(dnp no)
 		(property "Reference" "#PWR02"
-			(at 20.32 177.8 0)
+			(at 39.37 177.8 0)
 			(effects
 				(font
@@
 		)
 		(property "Value" "+5V"
-			(at 20.32 170.18 0)
+			(at 39.37 170.18 0)
 			(effects
 				(font
@@
 		)
 		(property "Footprint" ""
-			(at 20.32 173.99 0)
+			(at 39.37 173.99 0)
 			(effects
 				(font
@@
 		)
 		(property "Datasheet" ""
-			(at 20.32 173.99 0)
+			(at 39.37 173.99 0)
 			(effects
 				(font
@@
 		)
 		(property "Description" "Power symbol creates a global label with name \"+5V\""
-			(at 20.32 173.99 0)
+			(at 39.37 173.99 0)
 			(effects
 				(font

Commit message: fix LED order
Parts:
- D4: value LINE -> MIC
- D5: value MIC -> LINE
Changed lines of the file:
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@@
 	(title_block
 		(title "SW32 - Front Control Board")
-		(date "2024-05-30")
+		(date "2024-06-11")
 		(rev "1")
 		(company "saawsm")
@@
 			)
 		)
-		(property "Value" "MIC"
+		(property "Value" "LINE"
 			(at 154.686 24.384 0)
 			(effects
@@
 			)
 		)
-		(property "Value" "LINE"
+		(property "Value" "MIC"
 			(at 136.906 24.384 0)
 			(effects

Commit message: fix title block
Other:
- title: SW32 - Front Control Board -> SW32
Changed lines of the file:
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@@
 	(paper "A4")
 	(title_block
-		(title "SW32 - Front Control Board")
-		(date "2024-06-11")
+		(title "SW32")
+		(date "2024-06-12")
 		(rev "1")
 		(company "saawsm")
