File: kicad/output_board/output_board.kicad_pcb (KiCad board)
At the start: 2 copper layers, 109.2 x 48.3 mm, 88 parts, among them J1 DRV_PWR, J2 DRV, J3 CH_OUT, Q1 IRF9Z24NPBF, Q10 IRF9Z24NPBF, Q11 AO3400A, Q12 AO3400A, Q2 AO3400A, Q3 AO3400A, Q4 IRF9Z24NPBF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

Commit message: cleanup
Parts:
- moved C4 0.25 mm to (112.5, 75.3)
Routing:
- net GND: vias 37 -> 43
Changed lines of the file:
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@@
 		(locked yes)
 		(layer "F.Cu")
-		(at 112.520381 75.037197 90)
+		(at 112.522032 75.291197 90)
 		(descr "Capacitor SMD 0603 (1608 Metric), square (rectangular) end terminal, IPC_7351 nominal, (Body size source: IPC-SM-782 page 76, https://www.pcb-3d.com/wordpress/wp-content/uploads/ipc-sm-782a_amendment_1_and_2.pdf), generated with kicad-footprint-generator")
 		(tags "capacitor")
@@
 			(pinfunction "1")
 			(pintype "passive")
+			(zone_connect 2)
 		)
 		(pad "2" smd rect
@@
 			(pinfunction "2")
 			(pintype "passive")
+			(zone_connect 2)
 		)
 		(model "${KICAD8_3DMODEL_DIR}/Inductor_SMD.3dshapes/L_Sunlord_MWSA0603S.wrl"
@@
 			(pinfunction "K")
 			(pintype "passive")
+			(zone_connect 2)
 		)
 		(pad "2" smd roundrect
@@
 			(pinfunction "A")
 			(pintype "passive")
-			(thermal_bridge_width 0.5)
+			(zone_connect 2)
+			(thermal_bridge_width 1)
 		)
 		(model "${KICAD8_3DMODEL_DIR}/Diode_SMD.3dshapes/D_SMA.wrl"
@@
 			(pinfunction "GND")
 			(pintype "power_in")
+			(zone_connect 2)
 		)
 		(pad "7" smd rect
@@
 			(pinfunction "VIN")
 			(pintype "power_in")
+			(zone_connect 2)
 		)
 		(pad "8" smd rect
@@
 			(pinfunction "PH")
 			(pintype "output")
+			(zone_connect 2)
 		)
 		(pad "9" thru_hole circle
@@
 			(pinfunction "GNDPAD")
 			(pintype "power_in")
+			(zone_connect 2)
 		)
 		(pad "9" thru_hole circle
@@
 			(pinfunction "GNDPAD")
 			(pintype "power_in")
+			(zone_connect 2)
 		)
 		(pad "9" smd rect
@@
 			(pinfunction "GNDPAD")
 			(pintype "power_in")
+			(zone_connect 2)
 		)
 		(pad "9" smd rect
@@
 			(pinfunction "GNDPAD")
 			(pintype "power_in")
+			(zone_connect 2)
+			(thermal_bridge_width 1.5)
 		)
 		(pad "9" smd rect
@@
 			(pinfunction "GNDPAD")
 			(pintype "power_in")
+			(zone_connect 2)
 		)
 		(pad "9" thru_hole circle
@@
 			(pinfunction "GNDPAD")
 			(pintype "power_in")
+			(zone_connect 2)
 		)
 		(pad "9" thru_hole circle
@@
 			(pinfunction "GNDPAD")
 			(pintype "power_in")
+			(zone_connect 2)
 		)
 		(model "${KICAD8_3DMODEL_DIR}/Package_SO.3dshapes/HTSOP-8-1EP_3.9x4.9mm_Pitch1.27mm.wrl"
@@
 			(pinfunction "1")
 			(pintype "passive")
+			(zone_connect 2)
 		)
 	)
@@
 			(net 1 "GND")
 			(pintype "passive")
+			(zone_connect 2)
 		)
 		(pad "2" smd roundrect
@@
 			(net 2 "VIN")
 			(pintype "passive")
+			(zone_connect 2)
 		)
 		(model "${KICAD8_3DMODEL_DIR}/Capacitor_SMD.3dshapes/C_0805_2012Metric.wrl"
@@
 			(net 1 "GND")
 			(pintype "passive")
+			(zone_connect 2)
 		)
 		(pad "2" smd roundrect
@@
 			(net 2 "VIN")
 			(pintype "passive")
+			(zone_connect 2)
 		)
 		(model "${KICAD8_3DMODEL_DIR}/Capacitor_SMD.3dshapes/C_0805_2012Metric.wrl"
@@
 			(net 1 "GND")
 			(pintype "passive")
+			(zone_connect 2)
 		)
 		(pad "2" smd roundrect
@@
 			(net 2 "VIN")
 			(pintype "passive")
+			(zone_connect 2)
 		)
 		(model "${KICAD8_3DMODEL_DIR}/Capacitor_SMD.3dshapes/C_0805_2012Metric.wrl"
@@
 			(pinfunction "Pin_3")
 			(pintype "passive")
-			(thermal_bridge_width 0.5)
 		)
 		(pad "4" thru_hole oval
@@
 	)
 	(via
+		(at 125.222032 92.309197)
+		(size 0.8)
+		(drill 0.4)
+		(layers "F.Cu" "B.Cu")
+		(locked yes)
+		(free yes)
+		(net 1)
+	)
+	(via
+		(at 123.571032 93.706197)
+		(size 0.8)
+		(drill 0.4)
+		(layers "F.Cu" "B.Cu")
+		(locked yes)
+		(free yes)
+		(net 1)
+	)
+	(via
 		(at 120.523032 84.308197)
 		(size 0.8)
@@
 	)
 	(via
+		(at 122.795364 111.771122)
+		(size 0.6)
+		(drill 0.3)
+		(layers "F.Cu" "B.Cu")
+		(locked yes)
+		(free yes)
+		(net 1)
+	)
+	(via
 		(at 128.524032 97.008197)
 		(size 0.8)
@@
 	)
 	(via
+		(at 118.618032 88.880197)
+		(size 0.8)
+		(drill 0.4)
+		(layers "F.Cu" "B.Cu")
+		(locked yes)
+		(free yes)
+		(net 1)
+	)
+	(via
 		(at 128.524032 94.341197)
 		(size 0.8)
@@
 	)
 	(via
+		(at 110.357704 94.476794)
+		(size 0.8)
+		(drill 0.4)
+		(layers "F.Cu" "B.Cu")
+		(locked yes)
+		(free yes)
+		(net 1)
+	)
+	(via
 		(at 122.555032 83.292197)
 		(size 0.8)
@@
 	)
 	(via
+		(at 120.142032 87.610197)
+		(size 0.8)
+		(drill 0.4)
+		(layers "F.Cu" "B.Cu")
+		(locked yes)
+		(free yes)
+		(net 1)
+	)
+	(via
 		(at 115.443032 86.213197)
 		(size 0.8)
@@
 	)
 	(segment
-		(start 112.520381 75.812197)
+		(start 112.520381 76.067848)
 		(end 112.520381 79.756197)
 		(width 0.3)
@@
 	)
 	(segment
+		(start 112.522032 76.066197)
+		(end 112.520381 76.067848)
+		(width 0.3)
+		(locked yes)
+		(layer "F.Cu")
+		(net 3)
+	)
+	(segment
 		(start 145.897032 91.532871)
 		(end 146.209032 91.532871)
@@
 		(fill yes
 			(thermal_gap 0.2)
-			(thermal_bridge_width 0.5)
+			(thermal_bridge_width 0.3)
 		)
 		(polygon
 			(pts
-				(xy 116.967032 81.768197) (xy 116.967032 80.498197) (xy 120.777032 80.494957) (xy 120.777032 78.339197)
-				(xy 121.412032 78.339197) (xy 121.412032 71.989197) (xy 130.937032 71.989197) (xy 130.937032 81.768197)
+				(xy 120.523032 81.862305) (xy 120.142032 81.514197) (xy 116.967032 81.514197) (xy 116.967032 80.498197)
+				(xy 118.745032 80.498197) (xy 120.650032 77.704197) (xy 120.650032 71.989197) (xy 130.937032 71.989197)
+				(xy 130.937032 81.862305)
 			)
 		)
 	)
 	(zone
-		(net 1)
-		(net_name "GND")
+		(net 0)
+		(net_name "")
 		(locked yes)
 		(layer "F.Cu")
 		(hatch edge 0.5)
-		(priority 4)
 		(connect_pads
-			(clearance 0.2)
+			(clearance 0)
 		)
 		(min_thickness 0.2)
 		(filled_areas_thickness no)
-		(fill yes
-			(thermal_gap 0.2)
-			(thermal_bridge_width 1)
-		)
-		(polygon
-			(pts
-				(xy 114.300032 78.593197) (xy 116.078032 78.593197) (xy 116.078032 84.562197) (xy 114.300032 84.562197)
-			)
-		)
-	)
-	(zone
-		(net 4)
-		(net_name "Net-(D1-K)")
-		(locked yes)
-		(layer "F.Cu")
-		(hatch edge 0.5)
-		(priority 1)
-		(connect_pads
-			(clearance 0.2)
+		(keepout
+			(tracks allowed)
+			(vias allowed)
+			(pads allowed)
+			(copperpour not_allowed)
+			(footprints allowed)
 		)
-		(min_thickness 0.2)
-		(filled_areas_thickness no)
-		(fill yes
+		(fill
 			(thermal_gap 0.2)
 			(thermal_bridge_width 0.5)
@@
 		(polygon
 			(pts
-				(xy 116.967032 80.498197) (xy 116.967032 74.910197) (xy 110.109032 74.910197) (xy 110.109032 75.672197)
-				(xy 105.029032 75.672197) (xy 105.029032 71.989197) (xy 120.523032 71.989197) (xy 120.523032 80.494957)
+				(xy 113.499729 83.168893) (xy 111.633032 83.165197) (xy 111.633032 80.117197) (xy 113.499729 80.120893)
 			)
 		)
@@
 		(layer "F.Cu")
 		(hatch edge 0.5)
-		(priority 5)
+		(priority 1)
 		(connect_pads
-			(clearance 0.2)
+			(clearance 0.4)
 		)
 		(min_thickness 0.2)
@@
 		(fill yes
 			(thermal_gap 0.2)
-			(thermal_bridge_width 0.6)
+			(thermal_bridge_width 0.3)
 		)
 		(polygon
 			(pts
-				(xy 105.029032 71.989197) (xy 109.220032 71.989197) (xy 109.220032 75.672197) (xy 105.029032 75.672197)
+				(xy 116.967032 80.117197) (xy 116.967032 75.037197) (xy 105.029032 75.037197) (xy 105.029032 71.989197)
+				(xy 120.650032 71.989197) (xy 120.650032 77.704197) (xy 118.872032 80.113957)
 			)
 		)
@@
 		(polygon
 			(pts
-				(xy 102.997032 78.339197) (xy 111.379032 78.339197) (xy 111.35345 85.451013) (xy 108.176623 85.451197)
+				(xy 102.997032 78.339197) (xy 109.821381 78.339197) (xy 109.795799 85.451013) (xy 108.176623 85.451197)
 				(xy 108.204032 97.135197) (xy 102.997032 97.135197)
 			)
@@
 		(fill yes
 			(thermal_gap 0.2)
-			(thermal_bridge_width 0.5)
+			(thermal_bridge_width 0.3)
 		)
 		(polygon
@@
 			)
 		)
-	)
-	(zone
-		(net 1)
-		(net_name "GND")
-		(locked yes)
-		(layer "B.Cu")
-		(hatch edge 0.5)
-		(priority 4)
-		(connect_pads yes
-			(clearance 0.2)
-		)
-		(min_thickness 0.2)
-		(filled_areas_thickness no)
-		(fill yes
-			(thermal_gap 0.2)
-			(thermal_bridge_width 0.5)
-		)
-		(polygon
-			(pts
-				(xy 113.445644 78.613435) (xy 116.960219 78.627031) (xy 116.960219 84.596031) (xy 113.445644 84.582435)
-			)
-		)
