File: kicad/output_board/channel.kicad_sch (KiCad schematic)
At the start: 19 parts, among them Q4 IRF9Z24NPBF, Q5 AO3400A, Q6 AO3400A, T2 42TL004/42TU200, U2 LM324DT

Commit message: add capacitors
Parts:
- C11: renamed from C10; footprint (none) -> Capacitor_THT:CP_Radial_D8.0mm_P3.50mm; Service PCBA -> HandAssembly
- renumbered C12 to C13, C8 to C9
Changed lines of the file:
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@@
 	(title_block
 		(title "SW32 - Output Board")
-		(date "2024-05-26")
+		(date "2024-05-27")
 		(rev "1")
 		(company "saawsm")
@@
 		(on_board yes)
 		(dnp no)
-		(property "Reference" "#PWR022"
+		(property "Reference" "#PWR023"
 			(at 133.35 81.28 0)
 			(effects
@@
 			(project "output_board"
 				(path "/01334e4c-8cca-432b-91da-03bd5fdff467/997bb8f5-28c2-4cea-b91d-e0193d46d379"
-					(reference "#PWR022")
+					(reference "#PWR023")
 					(unit 1)
 				)
 				(path "/01334e4c-8cca-432b-91da-03bd5fdff467/784654d4-1031-4021-98e1-83b5de00916b"
-					(reference "#PWR030")
+					(reference "#PWR031")
 					(unit 1)
 				)
 				(path "/01334e4c-8cca-432b-91da-03bd5fdff467/7bfb3c86-2006-4e5a-a97d-386e3815f948"
-					(reference "#PWR038")
+					(reference "#PWR039")
 					(unit 1)
 				)
 				(path "/01334e4c-8cca-432b-91da-03bd5fdff467/1e63bddd-84c8-43db-b869-9e49fd6bc3cb"
-					(reference "#PWR046")
+					(reference "#PWR047")
 					(unit 1)
 				)
@@
 		(on_board yes)
 		(dnp no)
-		(property "Reference" "#PWR034"
+		(property "Reference" "#PWR035"
 			(at 212.09 113.03 0)
 			(effects
@@
 			(project "output_board"
 				(path "/01334e4c-8cca-432b-91da-03bd5fdff467/784654d4-1031-4021-98e1-83b5de00916b"
-					(reference "#PWR034")
+					(reference "#PWR035")
 					(unit 1)
 				)
 				(path "/01334e4c-8cca-432b-91da-03bd5fdff467/7bfb3c86-2006-4e5a-a97d-386e3815f948"
-					(reference "#PWR042")
+					(reference "#PWR043")
 					(unit 1)
 				)
 				(path "/01334e4c-8cca-432b-91da-03bd5fdff467/1e63bddd-84c8-43db-b869-9e49fd6bc3cb"
-					(reference "#PWR050")
+					(reference "#PWR051")
 					(unit 1)
 				)
 				(path "/01334e4c-8cca-432b-91da-03bd5fdff467/997bb8f5-28c2-4cea-b91d-e0193d46d379"
-					(reference "#PWR026")
+					(reference "#PWR027")
 					(unit 1)
 				)
@@
 		(on_board yes)
 		(dnp no)
-		(property "Reference" "#PWR023"
+		(property "Reference" "#PWR024"
 			(at 143.51 81.28 0)
 			(effects
@@
 			(project "output_board"
 				(path "/01334e4c-8cca-432b-91da-03bd5fdff467/997bb8f5-28c2-4cea-b91d-e0193d46d379"
-					(reference "#PWR023")
+					(reference "#PWR024")
 					(unit 1)
 				)
 				(path "/01334e4c-8cca-432b-91da-03bd5fdff467/784654d4-1031-4021-98e1-83b5de00916b"
-					(reference "#PWR031")
+					(reference "#PWR032")
 					(unit 1)
 				)
 				(path "/01334e4c-8cca-432b-91da-03bd5fdff467/7bfb3c86-2006-4e5a-a97d-386e3815f948"
-					(reference "#PWR039")
+					(reference "#PWR040")
 					(unit 1)
 				)
 				(path "/01334e4c-8cca-432b-91da-03bd5fdff467/1e63bddd-84c8-43db-b869-9e49fd6bc3cb"
-					(reference "#PWR047")
+					(reference "#PWR048")
 					(unit 1)
 				)
@@
 		(on_board yes)
 		(dnp no)
-		(property "Reference" "#PWR021"
+		(property "Reference" "#PWR022"
 			(at 60.96 147.32 0)
 			(effects
@@
 			(project "output_board"
 				(path "/01334e4c-8cca-432b-91da-03bd5fdff467/997bb8f5-28c2-4cea-b91d-e0193d46d379"
-					(reference "#PWR021")
+					(reference "#PWR022")
 					(unit 1)
 				)
 				(path "/01334e4c-8cca-432b-91da-03bd5fdff467/784654d4-1031-4021-98e1-83b5de00916b"
-					(reference "#PWR029")
+					(reference "#PWR030")
 					(unit 1)
 				)
 				(path "/01334e4c-8cca-432b-91da-03bd5fdff467/7bfb3c86-2006-4e5a-a97d-386e3815f948"
-					(reference "#PWR037")
+					(reference "#PWR038")
 					(unit 1)
 				)
 				(path "/01334e4c-8cca-432b-91da-03bd5fdff467/1e63bddd-84c8-43db-b869-9e49fd6bc3cb"
-					(reference "#PWR045")
+					(reference "#PWR046")
 					(unit 1)
 				)
@@
 		(on_board yes)
 		(dnp no)
-		(property "Reference" "#PWR027"
+		(property "Reference" "#PWR028"
 			(at 45.72 64.77 0)
 			(effects
@@
 			(project "output_board"
 				(path "/01334e4c-8cca-432b-91da-03bd5fdff467/784654d4-1031-4021-98e1-83b5de00916b"
-					(reference "#PWR027")
+					(reference "#PWR028")
 					(unit 1)
 				)
 				(path "/01334e4c-8cca-432b-91da-03bd5fdff467/7bfb3c86-2006-4e5a-a97d-386e3815f948"
-					(reference "#PWR035")
+					(reference "#PWR036")
 					(unit 1)
 				)
 				(path "/01334e4c-8cca-432b-91da-03bd5fdff467/1e63bddd-84c8-43db-b869-9e49fd6bc3cb"
-					(reference "#PWR043")
+					(reference "#PWR044")
 					(unit 1)
 				)
 				(path "/01334e4c-8cca-432b-91da-03bd5fdff467/997bb8f5-28c2-4cea-b91d-e0193d46d379"
-					(reference "#PWR019")
+					(reference "#PWR020")
 					(unit 1)
 				)
@@
 		(on_board yes)
 		(dnp no)
-		(property "Reference" "#PWR020"
+		(property "Reference" "#PWR021"
 			(at 45.72 80.01 0)
 			(effects
@@
 			(project "output_board"
 				(path "/01334e4c-8cca-432b-91da-03bd5fdff467/997bb8f5-28c2-4cea-b91d-e0193d46d379"
-					(reference "#PWR020")
+					(reference "#PWR021")
 					(unit 1)
 				)
 				(path "/01334e4c-8cca-432b-91da-03bd5fdff467/784654d4-1031-4021-98e1-83b5de00916b"
-					(reference "#PWR028")
+					(reference "#PWR029")
 					(unit 1)
 				)
 				(path "/01334e4c-8cca-432b-91da-03bd5fdff467/7bfb3c86-2006-4e5a-a97d-386e3815f948"
-					(reference "#PWR036")
+					(reference "#PWR037")
 					(unit 1)
 				)
 				(path "/01334e4c-8cca-432b-91da-03bd5fdff467/1e63bddd-84c8-43db-b869-9e49fd6bc3cb"
-					(reference "#PWR044")
+					(reference "#PWR045")
 					(unit 1)
 				)
@@
 		(dnp yes)
 		(fields_autoplaced yes)
-		(property "Reference" "C12"
+		(property "Reference" "C13"
 			(at 147.32 68.5799 0)
 			(effects
@@
 			(project "output_board"
 				(path "/01334e4c-8cca-432b-91da-03bd5fdff467/784654d4-1031-4021-98e1-83b5de00916b"
-					(reference "C12")
+					(reference "C13")
 					(unit 1)
 				)
 				(path "/01334e4c-8cca-432b-91da-03bd5fdff467/7bfb3c86-2006-4e5a-a97d-386e3815f948"
-					(reference "C15")
+					(reference "C16")
 					(unit 1)
 				)
 				(path "/01334e4c-8cca-432b-91da-03bd5fdff467/1e63bddd-84c8-43db-b869-9e49fd6bc3cb"
-					(reference "C18")
+					(reference "C19")
 					(unit 1)
 				)
 				(path "/01334e4c-8cca-432b-91da-03bd5fdff467/997bb8f5-28c2-4cea-b91d-e0193d46d379"
-					(reference "C9")
+					(reference "C10")
 					(unit 1)
 				)
@@
 		(on_board yes)
 		(dnp no)
-		(property "Reference" "C10"
+		(property "Reference" "C11"
 			(at 48.768 67.31 0)
 			(effects
@@
 			)
 		)
-		(property "Footprint" ""
+		(property "Footprint" "Capacitor_THT:CP_Radial_D8.0mm_P3.50mm"
 			(at 46.6852 72.39 0)
 			(effects
@@
 			)
 		)
-		(property "Service" "PCBA"
+		(property "Service" "HandAssembly"
 			(at 45.72 68.58 0)
 			(effects
@@
 			(project "output_board"
 				(path "/01334e4c-8cca-432b-91da-03bd5fdff467/784654d4-1031-4021-98e1-83b5de00916b"
-					(reference "C10")
+					(reference "C11")
 					(unit 1)
 				)
 				(path "/01334e4c-8cca-432b-91da-03bd5fdff467/7bfb3c86-2006-4e5a-a97d-386e3815f948"
-					(reference "C13")
+					(reference "C14")
 					(unit 1)
 				)
 				(path "/01334e4c-8cca-432b-91da-03bd5fdff467/1e63bddd-84c8-43db-b869-9e49fd6bc3cb"
-					(reference "C16")
+					(reference "C17")
 					(unit 1)
 				)
 				(path "/01334e4c-8cca-432b-91da-03bd5fdff467/997bb8f5-28c2-4cea-b91d-e0193d46d379"
-					(reference "C7")
+					(reference "C8")
 					(unit 1)
 				)
@@
 		(dnp no)
 		(fields_autoplaced yes)
-		(property "Reference" "C8"
+		(property "Reference" "C9"
 			(at 113.03 68.5799 0)
 			(effects
@@
 			(project "output_board"
 				(path "/01334e4c-8cca-432b-91da-03bd5fdff467/997bb8f5-28c2-4cea-b91d-e0193d46d379"
-					(reference "C8")
+					(reference "C9")
 					(unit 1)
 				)
 				(path "/01334e4c-8cca-432b-91da-03bd5fdff467/784654d4-1031-4021-98e1-83b5de00916b"
-					(reference "C11")
+					(reference "C12")
 					(unit 1)
 				)
 				(path "/01334e4c-8cca-432b-91da-03bd5fdff467/7bfb3c86-2006-4e5a-a97d-386e3815f948"
-					(reference "C14")
+					(reference "C15")
 					(unit 1)
 				)
 				(path "/01334e4c-8cca-432b-91da-03bd5fdff467/1e63bddd-84c8-43db-b869-9e49fd6bc3cb"
-					(reference "C17")
+					(reference "C18")
 					(unit 1)
 				)
@@
 		(on_board yes)
 		(dnp no)
-		(property "Reference" "#PWR025"
+		(property "Reference" "#PWR026"
 			(at 181.61 134.62 0)
 			(effects
@@
 			(project "output_board"
 				(path "/01334e4c-8cca-432b-91da-03bd5fdff467/997bb8f5-28c2-4cea-b91d-e0193d46d379"
-					(reference "#PWR025")
+					(reference "#PWR026")
 					(unit 1)
 				)
 				(path "/01334e4c-8cca-432b-91da-03bd5fdff467/784654d4-1031-4021-98e1-83b5de00916b"
-					(reference "#PWR033")
+					(reference "#PWR034")
 					(unit 1)
 				)
 				(path "/01334e4c-8cca-432b-91da-03bd5fdff467/7bfb3c86-2006-4e5a-a97d-386e3815f948"
-					(reference "#PWR041")
+					(reference "#PWR042")
 					(unit 1)
 				)
 				(path "/01334e4c-8cca-432b-91da-03bd5fdff467/1e63bddd-84c8-43db-b869-9e49fd6bc3cb"
-					(reference "#PWR049")
+					(reference "#PWR050")
 					(unit 1)
 				)
@@
 		(on_board yes)
 		(dnp no)
-		(property "Reference" "#PWR024"
+		(property "Reference" "#PWR025"
 			(at 165.1 60.96 0)
 			(effects
@@
 			(project "output_board"
 				(path "/01334e4c-8cca-432b-91da-03bd5fdff467/997bb8f5-28c2-4cea-b91d-e0193d46d379"
-					(reference "#PWR024")
+					(reference "#PWR025")
 					(unit 1)
 				)
 				(path "/01334e4c-8cca-432b-91da-03bd5fdff467/784654d4-1031-4021-98e1-83b5de00916b"
-					(reference "#PWR032")
+					(reference "#PWR033")
 					(unit 1)
 				)
 				(path "/01334e4c-8cca-432b-91da-03bd5fdff467/7bfb3c86-2006-4e5a-a97d-386e3815f948"
-					(reference "#PWR040")
+					(reference "#PWR041")
 					(unit 1)
 				)
 				(path "/01334e4c-8cca-432b-91da-03bd5fdff467/1e63bddd-84c8-43db-b869-9e49fd6bc3cb"
-					(reference "#PWR048")
+					(reference "#PWR049")
 					(unit 1)
 				)

Commit message: use 2x8 pin header
Parts:
- renumbered R11 to R10, R12 to R11, R22 to R21, R5 to R4, R6 to R5, R7 to R6, R8 to R7, R9 to R8, R10 to R9
Connections:
- net OUTA: now also T2.4 (S1); no longer T2.6 (S2)
- net OUTB: now also T2.6 (S2); no longer T2.4 (S1)

Commit message: add draft output board
Parts:
- removed C13: 100nF, Capacitor_SMD:C_0603_1608Metric, symbol Device:C
- removed R8: 1k, Resistor_SMD:R_0603_1608Metric, symbol Device:R
- renumbered C11 to C10, R11 to R10, R21 to R19, R9 to R8, R10 to R9

Commit message: fix title block
Other:
- title: SW32 - Output Board -> SW32
Changed lines of the file:
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@@
 	(paper "A4")
 	(title_block
-		(title "SW32 - Output Board")
-		(date "2024-06-01")
+		(title "SW32")
+		(date "2024-06-12")
 		(rev "1")
 		(company "saawsm")
