File: kicad/front_panel/front_panel.kicad_sch (KiCad schematic)
At the start: 8 parts

Commit message: fix title block
Other:
- title: SW32 - Front Panel -> SW32
Changed lines of the file:
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@@
 	(paper "A4")
 	(title_block
-		(title "SW32 - Front Panel")
-		(date "2024-05-27")
+		(title "SW32")
+		(date "2024-06-12")
 		(rev "1")
 		(company "saawsm")
