File: kicad/front_panel/front_panel.kicad_pcb (KiCad board)
At the start: 2 copper layers, 203.2 x 70.2 mm, 8 parts

Commit message: add plot settings
Other:
- board text added: "${TITLE} ${PROJECTNAME} rev${REVISION}"
- board text removed: "${TITLE} ${PROJECTNAME} rev${REVISION} ${hash}"
Changed lines of the file:
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@@
 			(plot_on_all_layers_selection 0x0000000_00000000)
 			(disableapertmacros no)
-			(usegerberextensions no)
-			(usegerberattributes yes)
-			(usegerberadvancedattributes yes)
-			(creategerberjobfile yes)
+			(usegerberextensions yes)
+			(usegerberattributes no)
+			(usegerberadvancedattributes no)
+			(creategerberjobfile no)
 			(dashed_line_dash_ratio 12.000000)
 			(dashed_line_gap_ratio 3.000000)
@@
 			(plotinvisibletext no)
 			(sketchpadsonfab no)
-			(subtractmaskfromsilk no)
+			(subtractmaskfromsilk yes)
 			(outputformat 1)
 			(mirror no)
-			(drillshape 1)
+			(drillshape 0)
 			(scaleselection 1)
-			(outputdirectory "")
+			(outputdirectory "../../pcb/front_panel/")
 		)
 	)
@@
 		(layer "Edge.Cuts")
 	)
-	(gr_text "${TITLE}\n${PROJECTNAME}\nrev${REVISION} ${hash}"
+	(gr_text "${TITLE}\n${PROJECTNAME}\nrev${REVISION}"
 		(locked yes)
 		(at 180.34 82.55 0)
